File: KiCad/RDAT/RDAT.kicad_pcb (KiCad board)
At the start: 2 copper layers, 49.6 x 53.5 mm, 2 parts

Commit message: Push before Board Layout
Parts:
- removed REF**: SMTWE2015MTJ, Mounting_Wuerth:Mounting_Wuerth_WA-SMSI-M2_H1.5mm_9774015243
- removed REF**: LattePanda_Module_H4.0mm_Horizontal, footprints:LattePanda_Module_H4.0mm_Horizontal
Other:
- board outline removed

Commit message: placed board components, with errors
Parts:
- added A1: LattePanda_Mu, footprints:LattePanda_Module_H4.0mm_Horizontal, F.Cu at (-66.5, -75.2)
- added ACFET1: SI7617DN-T1-GE3, footprints:POWERPAK_1212-8_VIS, F.Cu at (-44.8, 95.2)
- added ACFET2: SI7617DN-T1-GE3, footprints:POWERPAK_1212-8_VIS, F.Cu at (-44.8, 100.3)
- added BATFET1: SI7617DN-T1-GE3, footprints:POWERPAK_1212-8_VIS, F.Cu at (-44.8, 105.4)
- added BT1: 54, footprints:BAT_BK-18650-CLIP, F.Cu at (-96.5, 20.0)
- added BT10: 54, footprints:BAT_BK-18650-CLIP, F.Cu at (-82.0, 60.4)
- added BT11: 54, footprints:BAT_BK-18650-CLIP, F.Cu at (-67.5, 60.4)
- added BT12: 54, footprints:BAT_BK-18650-CLIP, F.Cu at (-53.0, 60.4)
- added BT13: 54, footprints:BAT_BK-18650-CLIP, F.Cu at (-96.5, 80.6)
- added BT14: 54, footprints:BAT_BK-18650-CLIP, F.Cu at (-82.0, 80.6)
- added BT15: 54, footprints:BAT_BK-18650-CLIP, F.Cu at (-67.5, 80.6)
- added BT16: 54, footprints:BAT_BK-18650-CLIP, F.Cu at (-53.0, 80.6)
- added BT17: 3v, footprints:HARWIN_S8411-45R, F.Cu at (-95.6, -3.06)
- added BT2: 54, footprints:BAT_BK-18650-CLIP, F.Cu at (-82.0, 20.0)
- added BT3: 54, footprints:BAT_BK-18650-CLIP, F.Cu at (-67.5, 20.0)
- added BT4: 54, footprints:BAT_BK-18650-CLIP, F.Cu at (-53.0, 20.0)
- added BT5: 54, footprints:BAT_BK-18650-CLIP, F.Cu at (-96.5, 40.2)
- added BT6: 54, footprints:BAT_BK-18650-CLIP, F.Cu at (-82.0, 40.2)
- added BT7: 54, footprints:BAT_BK-18650-CLIP, F.Cu at (-67.5, 40.2)
- added BT8: 54, footprints:BAT_BK-18650-CLIP, F.Cu at (-53.0, 40.2)
- added BT9: 54, footprints:BAT_BK-18650-CLIP, F.Cu at (-96.5, 60.4)
- added C1: 100n, Capacitor_SMD:C_0402_1005Metric, F.Cu at (-186.1, 48.6)
- added C10: 100n, Capacitor_SMD:C_0402_1005Metric, F.Cu at (-183.2, 56.4)
- added C11: 100n, Capacitor_SMD:C_0402_1005Metric, F.Cu at (-180.3, 48.6)
- added C12: 100n, Capacitor_SMD:C_0402_1005Metric, F.Cu at (-180.3, 50.5)
- added C13: 15p, Capacitor_SMD:C_0402_1005Metric, F.Cu at (-180.3, 52.5)
- added C14: 15p, Capacitor_SMD:C_0402_1005Metric, F.Cu at (-180.3, 54.5)
- added C15: 1uF, Capacitor_SMD:C_0402_1005Metric, F.Cu at (-37.9, 51.9)
- added C16: 1uF, Capacitor_SMD:C_0402_1005Metric, F.Cu at (-37.9, 53.8)
- added C17: 1uF/10%, Capacitor_SMD:C_0402_1005Metric, F.Cu at (-37.9, 55.8)
- added C18: 22uF/6.3V, Capacitor_SMD:C_0402_1005Metric, F.Cu at (-37.9, 22.1)
- added C19: 10uF/6.3v, Capacitor_SMD:C_0402_1005Metric, F.Cu at (-37.9, 24.1)
- added C2: 100n, Capacitor_SMD:C_0402_1005Metric, F.Cu at (-186.1, 50.5)
- added C20: 0.1uF/16v, Capacitor_SMD:C_0402_1005Metric, F.Cu at (-37.9, 26.1)
- added C21: 0.1uF/16v, Capacitor_SMD:C_0402_1005Metric, F.Cu at (-37.9, 28.1)
- added C22: 100nF/64mOhm, Capacitor_SMD:C_0402_1005Metric, F.Cu at (-204.2, 83.7)
- added C23: 47uF/3.037mOhm, Capacitor_SMD:C_1210_3225Metric, F.Cu at (-201.8, 98.8)
- added C24: 100nF/50V, Capacitor_SMD:C_0402_1005Metric, F.Cu at (-31.9, 76.3)
- added C25: 100nF/50V, Capacitor_SMD:C_0402_1005Metric, F.Cu at (-97.4, 124.8)
- added C26: 100nF/50V, Capacitor_SMD:C_0402_1005Metric, F.Cu at (-97.4, 126.8)
- added C27: 100nF/50V, Capacitor_SMD:C_0402_1005Metric, F.Cu at (-97.4, 128.8)
- added C28: 100nF/50V, Capacitor_SMD:C_0402_1005Metric, F.Cu at (-94.5, 124.8)
- added C29: 100nF/50V, Capacitor_SMD:C_0402_1005Metric, F.Cu at (-94.5, 126.8)
- added C3: 1u, Capacitor_SMD:C_0402_1005Metric, F.Cu at (-186.1, 52.5)
- added C30: 100nF/50V, Capacitor_SMD:C_0402_1005Metric, F.Cu at (-94.5, 128.8)
- added C31: 100nF/50V, Capacitor_SMD:C_0402_1005Metric, F.Cu at (-91.7, 124.8)
- added C32: 100nF/64mOhm, Capacitor_SMD:C_0402_1005Metric, F.Cu at (-204.2, 85.7)
- added C33: 1uF, footprints:CAP-SMD_BD4.0-L4.3-W4.3-FD, F.Cu at (-44.4, 110.7)
- added C34: 0.1uF, Capacitor_SMD:C_0402_1005Metric, F.Cu at (-65.8, 117.4)
- added C35: 0.1uF, Capacitor_SMD:C_0402_1005Metric, F.Cu at (-65.8, 119.4)
- added C36: 1uF, Capacitor_SMD:C_0402_1005Metric, F.Cu at (-65.8, 121.3)
- added C37: 0.1uF, Capacitor_SMD:C_0402_1005Metric, F.Cu at (-65.8, 123.3)
- added C38: 0.1uF, Capacitor_SMD:C_0402_1005Metric, F.Cu at (-65.8, 125.3)
- added C39: 0.1uF, Capacitor_SMD:C_0402_1005Metric, F.Cu at (-62.9, 117.4)
- added C4: 100n, Capacitor_SMD:C_0402_1005Metric, F.Cu at (-186.1, 54.5)
- added C40: 10uF, Capacitor_SMD:C_0402_1005Metric, F.Cu at (-62.9, 119.4)
- added C41: 10uF, Capacitor_SMD:C_0402_1005Metric, F.Cu at (-62.9, 121.3)
- added C42: 22pF, Capacitor_SMD:C_0402_1005Metric, F.Cu at (-62.9, 123.3)
- added C43: 1uF, footprints:CAP-SMD_BD4.0-L4.3-W4.3-FD, F.Cu at (-44.4, 116.3)
- added C44: 0.1uF, Capacitor_SMD:C_0402_1005Metric, F.Cu at (-62.9, 125.3)
- added C45: 10uF, footprints:CAP-SMD_BD6.3-L6.6-W6.6-LS7.4-FD, F.Cu at (-62.3, 96.6)
- added C46: 10uF, footprints:CAP-SMD_BD6.3-L6.6-W6.6-LS7.4-FD, F.Cu at (-62.3, 104.6)
- added C47: 1uF, Capacitor_SMD:C_0402_1005Metric, F.Cu at (-60.0, 117.4)
- added C48: 47uF/3.037mOhm, Capacitor_SMD:C_1210_3225Metric, F.Cu at (-201.8, 103.0)
- added C49: 2.2uF, footprints:CAP-SMD_BD6.3-L6.6-W6.6-LS7.4-FD, F.Cu at (-62.3, 112.5)
- added C5: 1u, Capacitor_SMD:C_0402_1005Metric, F.Cu at (-186.1, 56.4)
- added C50: 22uF, Capacitor_SMD:C_0805_2012Metric, F.Cu at (-43.5, 11.4)
- added C51: 22uF/10V, Capacitor_SMD:C_0402_1005Metric, F.Cu at (-186.0, 104.8)
- added C52: 270pF, Capacitor_SMD:C_0201_0603Metric, F.Cu at (-227.1, 110.8)
- added C53: 12nF, Capacitor_SMD:C_0402_1005Metric, F.Cu at (-204.2, 87.7)
- added C54: 470nF, Capacitor_SMD:C_0402_1005Metric, F.Cu at (-204.2, 89.6)
- added C55: 100nF, Capacitor_SMD:C_0402_1005Metric, F.Cu at (-204.2, 91.6)
- added C56: 0.1uF/16v, Capacitor_SMD:C_0402_1005Metric, F.Cu at (-37.9, 30.0)
- added C57: 1uF/6.3v, Capacitor_SMD:C_0402_1005Metric, F.Cu at (-37.9, 32.0)
- added C58: 1uF/10%, Capacitor_SMD:C_0402_1005Metric, F.Cu at (-37.9, 57.8)
- added C59: 1uF/10%, Capacitor_SMD:C_0402_1005Metric, F.Cu at (-37.9, 59.7)
- added C6: 100n, Capacitor_SMD:C_0402_1005Metric, F.Cu at (-183.2, 48.6)
- added C60: 10uF/1mOhm, Capacitor_SMD:C_0402_1005Metric, F.Cu at (-204.2, 93.6)
- added C61: 4.7uF/3.52mohm(ESR), Capacitor_SMD:C_0402_1005Metric, F.Cu at (-201.3, 83.7)
- added C62: 1uF/10%, Capacitor_SMD:C_0402_1005Metric, F.Cu at (-35.0, 51.9)
- added C63: 1uF/10%, Capacitor_SMD:C_0402_1005Metric, F.Cu at (-35.0, 53.8)
- added C64: 0.1uF, Capacitor_SMD:C_0402_1005Metric, F.Cu at (-35.0, 55.8)
- added C65: 0.1uF, Capacitor_SMD:C_0402_1005Metric, F.Cu at (-35.0, 57.8)
- added C66: 1uF/16V, Capacitor_SMD:C_0402_1005Metric, F.Cu at (-201.3, 85.7)
- added C67: 0.1uF, Capacitor_SMD:C_0402_1005Metric, F.Cu at (-35.0, 59.7)
- added C68: 100fP/50v, Capacitor_SMD:C_0402_1005Metric, F.Cu at (-37.9, 34.0)
- added C69: 1uF/16V, Capacitor_SMD:C_0402_1005Metric, F.Cu at (-201.3, 87.7)
- added C7: 100n, Capacitor_SMD:C_0402_1005Metric, F.Cu at (-183.2, 50.5)
- added C70: 47pF/0Ohm, Capacitor_SMD:C_0402_1005Metric, F.Cu at (-201.3, 89.6)
- added C71: 47uF/3.037mOhm, Capacitor_SMD:C_1210_3225Metric, F.Cu at (-201.8, 107.3)
- added C72: 82pF/0Ohm, Capacitor_SMD:C_0201_0603Metric, F.Cu at (-227.1, 112.6)
- added C78: 1uF/16V, Capacitor_SMD:C_0402_1005Metric, F.Cu at (-148.1, 106.9)
- added C79: 0.1uF, Capacitor_SMD:C_0402_1005Metric, F.Cu at (-60.0, 119.4)
- added C8: 100n, Capacitor_SMD:C_0402_1005Metric, F.Cu at (-183.2, 52.5)
- added C80: 220nF/50V, Capacitor_SMD:C_0402_1005Metric, F.Cu at (-193.6, 112.7)
- added C81: 220nF/50V, Capacitor_SMD:C_0402_1005Metric, F.Cu at (-193.6, 114.7)
- added C82: 10uF/10V, Capacitor_SMD:C_0402_1005Metric, F.Cu at (-193.6, 116.7)
- added C83: 100nF/50V, Capacitor_SMD:C_0402_1005Metric, F.Cu at (-193.6, 118.6)
- added C84: 10uF/10V, Capacitor_SMD:C_0402_1005Metric, F.Cu at (-193.6, 120.6)
- added C85: 100nF/50V, Capacitor_SMD:C_0402_1005Metric, F.Cu at (-193.6, 122.6)
- added C9: 100n, Capacitor_SMD:C_0402_1005Metric, F.Cu at (-183.2, 54.5)
- added C91: 100nF/50V, Capacitor_SMD:C_0402_1005Metric, F.Cu at (-91.7, 126.8)
- added C92: 100nF/50V, Capacitor_SMD:C_0402_1005Metric, F.Cu at (-91.7, 128.8)
- added CTTC1: 47nF, Capacitor_SMD:C_0402_1005Metric, F.Cu at (-60.0, 121.3)
- added C_{OUT}1: 10uF, Capacitor_SMD:C_0402_1005Metric, F.Cu at (-201.3, 91.6)
- added Ccomp3: 1.8nF, Capacitor_SMD:C_0402_1005Metric, F.Cu at (-201.3, 93.6)
- added Cin1: 4.7uF, Capacitor_SMD:C_0402_1005Metric, F.Cu at (-198.4, 83.7)
- added Css1: 3.3nF, Capacitor_SMD:C_0402_1005Metric, F.Cu at (-198.4, 85.7)
- added Cvcc1: 1uF, Capacitor_SMD:C_1206_3216Metric, F.Cu at (-225.5, 108.3)
- added D1: Diode, Diode_SMD:D_MiniMELF, F.Cu at (-229.0, 32.3)
- added D10: Diode, Diode_SMD:D_MiniMELF, F.Cu at (-229.0, 62.4)
- added D100: Diode, Diode_SMD:D_MiniMELF, F.Cu at (-190.7, 62.4)
- added D101: Diode, Diode_SMD:D_MiniMELF, F.Cu at (-190.7, 65.7)
- added D102: Diode, Diode_SMD:D_MiniMELF, F.Cu at (-190.7, 69.0)
- added D103: Diode, Diode_SMD:D_MiniMELF, F.Cu at (-190.7, 72.4)
- added D104: Diode, Diode_SMD:D_MiniMELF, F.Cu at (-190.7, 75.7)
- added D105: SD05_SOD323, Diode_SMD:D_SOD-323, F.Cu at (-22.7, 22.6)
- added D106: SD05_SOD323, Diode_SMD:D_SOD-323, F.Cu at (-22.7, 25.6)
- added D109: 1N5819WS, Diode_SMD:D_SOD-323, F.Cu at (-31.2, 73.8)
- added D11: Diode, Diode_SMD:D_MiniMELF, F.Cu at (-229.0, 65.7)
- added D110: ESD5V0B03, Diode_SMD:D_SOD-882, F.Cu at (-88.7, 113.1)
- added D111: BAT54J, Diode_SMD:D_SOD-323F, F.Cu at (-33.0, 114.4)
- added D112: LED, Diode_SMD:D_1206_3216Metric, F.Cu at (-38.0, 109.6)
- added D113: LED, Diode_SMD:D_1206_3216Metric, F.Cu at (-38.0, 113.0)
- added D114: LED, Diode_SMD:D_1206_3216Metric, F.Cu at (-38.0, 116.4)
- added D116: LED_G, LED_SMD:LED_0603_1608Metric, F.Cu at (-206.7, 111.1)
- added D118: ESD5V0B03, Diode_SMD:D_SOD-882, F.Cu at (-88.7, 115.4)
- added D119: ESD9B5.0ST5G, Diode_SMD:D_SOD-923, F.Cu at (-26.1, 22.1)
- added D12: Diode, Diode_SMD:D_MiniMELF, F.Cu at (-229.0, 69.0)
- added D120: ESD9B5.0ST5G, Diode_SMD:D_SOD-923, F.Cu at (-26.1, 24.1)
- added D121: ESD9B5.0ST5G, Diode_SMD:D_SOD-923, F.Cu at (-26.1, 26.0)
- added D122: ESD9B5.0ST5G, Diode_SMD:D_SOD-923, F.Cu at (-26.1, 28.0)
- added D123: ESD5V0B03, Diode_SMD:D_SOD-882, F.Cu at (-88.7, 117.8)
- added D124: ESD5V0B03, Diode_SMD:D_SOD-882, F.Cu at (-157.0, 101.1)
- added D125: ESD5V0B03, Diode_SMD:D_SOD-882, F.Cu at (-157.0, 103.5)
- added D126: PESD24VS1UL-N, Diode_SMD:D_SOD-882, F.Cu at (-157.0, 105.8)
- added D127: PESD24VS1UL-N, Diode_SMD:D_SOD-882, F.Cu at (-157.0, 108.1)
- added D128: PESD24VS1UL-N, Diode_SMD:D_SOD-882, F.Cu at (-157.0, 110.5)
- added D129: ESD5V0B03, Diode_SMD:D_SOD-882, F.Cu at (-198.4, 110.6)
- added D13: Diode, Diode_SMD:D_MiniMELF, F.Cu at (-229.0, 72.4)
- added D130: 1N5819WS, Diode_SMD:D_SOD-323, F.Cu at (-76.9, 113.4)
- added D131: ESD5V0B03, Diode_SMD:D_SOD-882, F.Cu at (-198.4, 112.9)
- added D14: Diode, Diode_SMD:D_MiniMELF, F.Cu at (-229.0, 75.7)
- added D15: Diode, Diode_SMD:D_MiniMELF, F.Cu at (-229.0, 79.1)
- added D16: Diode, Diode_SMD:D_MiniMELF, F.Cu at (-222.6, 32.3)
- added D17: Diode, Diode_SMD:D_MiniMELF, F.Cu at (-222.6, 35.6)
- added D18: Diode, Diode_SMD:D_MiniMELF, F.Cu at (-222.6, 39.0)
- added D19: Diode, Diode_SMD:D_MiniMELF, F.Cu at (-222.6, 42.3)
- added D2: Diode, Diode_SMD:D_MiniMELF, F.Cu at (-229.0, 35.6)
- added D20: Diode, Diode_SMD:D_MiniMELF, F.Cu at (-222.6, 45.7)
- added D21: Diode, Diode_SMD:D_MiniMELF, F.Cu at (-222.6, 49.0)
- added D22: Diode, Diode_SMD:D_MiniMELF, F.Cu at (-222.6, 52.3)
- added D23: Diode, Diode_SMD:D_MiniMELF, F.Cu at (-222.6, 55.7)
- added D24: Diode, Diode_SMD:D_MiniMELF, F.Cu at (-222.6, 59.0)
- added D25: Diode, Diode_SMD:D_MiniMELF, F.Cu at (-222.6, 62.4)
- added D26: Diode, Diode_SMD:D_MiniMELF, F.Cu at (-222.6, 65.7)
- added D27: Diode, Diode_SMD:D_MiniMELF, F.Cu at (-222.6, 69.0)
- added D28: Diode, Diode_SMD:D_MiniMELF, F.Cu at (-222.6, 72.4)
- added D29: Diode, Diode_SMD:D_MiniMELF, F.Cu at (-222.6, 75.7)
- added D3: Diode, Diode_SMD:D_MiniMELF, F.Cu at (-229.0, 39.0)
- added D30: Diode, Diode_SMD:D_MiniMELF, F.Cu at (-222.6, 79.1)
- added D31: Diode, Diode_SMD:D_MiniMELF, F.Cu at (-216.2, 32.3)
- added D32: Diode, Diode_SMD:D_MiniMELF, F.Cu at (-216.2, 35.6)
- added D33: Diode, Diode_SMD:D_MiniMELF, F.Cu at (-216.2, 39.0)
- added D34: Diode, Diode_SMD:D_MiniMELF, F.Cu at (-216.2, 42.3)
- added D35: Diode, Diode_SMD:D_MiniMELF, F.Cu at (-216.2, 45.7)
- added D36: Diode, Diode_SMD:D_MiniMELF, F.Cu at (-216.2, 49.0)
- added D37: Diode, Diode_SMD:D_MiniMELF, F.Cu at (-216.2, 52.3)
- added D38: Diode, Diode_SMD:D_MiniMELF, F.Cu at (-216.2, 55.7)
- added D39: Diode, Diode_SMD:D_MiniMELF, F.Cu at (-216.2, 59.0)
- added D4: Diode, Diode_SMD:D_MiniMELF, F.Cu at (-229.0, 42.3)
- added D40: Diode, Diode_SMD:D_MiniMELF, F.Cu at (-216.2, 62.4)
- added D41: Diode, Diode_SMD:D_MiniMELF, F.Cu at (-216.2, 65.7)
- added D42: Diode, Diode_SMD:D_MiniMELF, F.Cu at (-216.2, 69.0)
- added D43: Diode, Diode_SMD:D_MiniMELF, F.Cu at (-216.2, 72.4)
- added D44: Diode, Diode_SMD:D_MiniMELF, F.Cu at (-216.2, 75.7)
- added D45: Diode, Diode_SMD:D_MiniMELF, F.Cu at (-216.2, 79.1)
- added D46: Diode, Diode_SMD:D_MiniMELF, F.Cu at (-209.8, 32.3)
- added D47: Diode, Diode_SMD:D_MiniMELF, F.Cu at (-209.8, 35.6)
- added D48: Diode, Diode_SMD:D_MiniMELF, F.Cu at (-209.8, 39.0)
- added D49: Diode, Diode_SMD:D_MiniMELF, F.Cu at (-209.8, 42.3)
- added D5: Diode, Diode_SMD:D_MiniMELF, F.Cu at (-229.0, 45.7)
- added D50: Diode, Diode_SMD:D_MiniMELF, F.Cu at (-209.8, 45.7)
- added D51: Diode, Diode_SMD:D_MiniMELF, F.Cu at (-209.8, 49.0)
- added D52: Diode, Diode_SMD:D_MiniMELF, F.Cu at (-209.8, 52.3)
- added D53: Diode, Diode_SMD:D_MiniMELF, F.Cu at (-209.8, 55.7)
- added D54: Diode, Diode_SMD:D_MiniMELF, F.Cu at (-209.8, 59.0)
- added D55: Diode, Diode_SMD:D_MiniMELF, F.Cu at (-209.8, 62.4)
- added D56: Diode, Diode_SMD:D_MiniMELF, F.Cu at (-209.8, 65.7)
- added D57: Diode, Diode_SMD:D_MiniMELF, F.Cu at (-209.8, 69.0)
- added D58: Diode, Diode_SMD:D_MiniMELF, F.Cu at (-209.8, 72.4)
- added D59: Diode, Diode_SMD:D_MiniMELF, F.Cu at (-209.8, 75.7)
- added D6: Diode, Diode_SMD:D_MiniMELF, F.Cu at (-229.0, 49.0)
- added D60: Diode, Diode_SMD:D_MiniMELF, F.Cu at (-209.8, 79.1)
- added D61: Diode, Diode_SMD:D_MiniMELF, F.Cu at (-203.5, 32.3)
- added D62: Diode, Diode_SMD:D_MiniMELF, F.Cu at (-203.5, 35.6)
- added D63: Diode, Diode_SMD:D_MiniMELF, F.Cu at (-203.5, 39.0)
- added D64: Diode, Diode_SMD:D_MiniMELF, F.Cu at (-203.5, 42.3)
- added D65: Diode, Diode_SMD:D_MiniMELF, F.Cu at (-203.5, 45.7)
- added D66: Diode, Diode_SMD:D_MiniMELF, F.Cu at (-203.5, 49.0)
- added D67: Diode, Diode_SMD:D_MiniMELF, F.Cu at (-203.5, 52.3)
- added D68: Diode, Diode_SMD:D_MiniMELF, F.Cu at (-203.5, 55.7)
- added D69: Diode, Diode_SMD:D_MiniMELF, F.Cu at (-203.5, 59.0)
- added D7: Diode, Diode_SMD:D_MiniMELF, F.Cu at (-229.0, 52.3)
- added D70: Diode, Diode_SMD:D_MiniMELF, F.Cu at (-203.5, 62.4)
- added D71: Diode, Diode_SMD:D_MiniMELF, F.Cu at (-203.5, 65.7)
- added D72: Diode, Diode_SMD:D_MiniMELF, F.Cu at (-203.5, 69.0)
- added D73: Diode, Diode_SMD:D_MiniMELF, F.Cu at (-203.5, 72.4)
- added D74: Diode, Diode_SMD:D_MiniMELF, F.Cu at (-203.5, 75.7)
- added D75: Diode, Diode_SMD:D_MiniMELF, F.Cu at (-203.5, 79.1)
- added D76: Diode, Diode_SMD:D_MiniMELF, F.Cu at (-197.1, 32.3)
- added D77: Diode, Diode_SMD:D_MiniMELF, F.Cu at (-197.1, 35.6)
- added D78: Diode, Diode_SMD:D_MiniMELF, F.Cu at (-197.1, 39.0)
- added D79: Diode, Diode_SMD:D_MiniMELF, F.Cu at (-197.1, 42.3)
- added D8: Diode, Diode_SMD:D_MiniMELF, F.Cu at (-229.0, 55.7)
- added D80: Diode, Diode_SMD:D_MiniMELF, F.Cu at (-197.1, 45.7)
- added D81: Diode, Diode_SMD:D_MiniMELF, F.Cu at (-197.1, 49.0)
- added D82: Diode, Diode_SMD:D_MiniMELF, F.Cu at (-197.1, 52.3)
- added D83: Diode, Diode_SMD:D_MiniMELF, F.Cu at (-197.1, 55.7)
- added D84: Diode, Diode_SMD:D_MiniMELF, F.Cu at (-197.1, 59.0)
- added D85: Diode, Diode_SMD:D_MiniMELF, F.Cu at (-197.1, 62.4)
- added D86: Diode, Diode_SMD:D_MiniMELF, F.Cu at (-197.1, 65.7)
- added D87: Diode, Diode_SMD:D_MiniMELF, F.Cu at (-197.1, 69.0)
- added D88: Diode, Diode_SMD:D_MiniMELF, F.Cu at (-197.1, 72.4)
- added D89: Diode, Diode_SMD:D_MiniMELF, F.Cu at (-197.1, 75.7)
- added D9: Diode, Diode_SMD:D_MiniMELF, F.Cu at (-229.0, 59.0)
- added D90: Diode, Diode_SMD:D_MiniMELF, F.Cu at (-197.1, 79.1)
- added D91: Diode, Diode_SMD:D_MiniMELF, F.Cu at (-190.7, 32.3)
- added D92: Diode, Diode_SMD:D_MiniMELF, F.Cu at (-190.7, 35.6)
- added D93: Diode, Diode_SMD:D_MiniMELF, F.Cu at (-190.7, 39.0)
- added D94: Diode, Diode_SMD:D_MiniMELF, F.Cu at (-190.7, 42.3)
- added D95: Diode, Diode_SMD:D_MiniMELF, F.Cu at (-190.7, 45.7)
- added D96: Diode, Diode_SMD:D_MiniMELF, F.Cu at (-190.7, 49.0)
- added D97: Diode, Diode_SMD:D_MiniMELF, F.Cu at (-190.7, 52.3)
- added D98: Diode, Diode_SMD:D_MiniMELF, F.Cu at (-190.7, 55.7)
- added D99: Diode, Diode_SMD:D_MiniMELF, F.Cu at (-190.7, 59.0)
- added F1: 6V/50mA, Fuse:Fuse_0805_2012Metric, F.Cu at (-81.3, 113.4)
- added F2: 6V/1A, Fuse:Fuse_0805_2012Metric, F.Cu at (-192.8, 105.3)
- added F3: 6V/1A, Fuse:Fuse_0805_2012Metric, F.Cu at (-192.8, 108.3)
- added H5: MountingHole_Pad, MountingHole:MountingHole_2.2mm_M2_Pad_TopBottom, F.Cu at (-84.5, -11.5)
- added H6: MountingHole_Pad, MountingHole:MountingHole_2.2mm_M2_Pad_TopBottom, F.Cu at (-84.5, -5.59)
- added H8: MountingHole_M2.0, MountingHole:MountingHole_2.2mm_M2_Pad_TopBottom, F.Cu at (-186.2, 126.0)
- added J1: Conn_01x02, Connector_PinHeader_1.00mm:PinHeader_1x02_P1.00mm_Vertical, F.Cu at (-175.3, 41.3)
- added J16: MDT420E03001, footprints:AMPHENOL_MDT420E03001, F.Cu at (-180.4, 119.2)
- added J18: MUSBRM1C130, footprints:AMPHENOL_MUSBRM1C130, F.Cu at (-145.9, 87.3)
- added J2: Conn_01x02, Connector_PinHeader_1.00mm:PinHeader_1x02_P1.00mm_Vertical, F.Cu at (-172.0, 41.3)
- added J3: Conn_01x02, Connector_PinHeader_1.00mm:PinHeader_1x02_P1.00mm_Vertical, F.Cu at (-18.9, 22.7)
- added J4: Bus_M.2_Socket_B, footprints:AMPHENOL_MDT420B03001, F.Cu at (-27.5, 17.1)
- added J5: USB_A_Stacked, footprints:CONN8_MUSBC_1211x569_AMP, F.Cu at (-179.6, 94.9)
- added J6: HDMI_A, footprints:AMPHENOL_MHDRA111M0, F.Cu at (-87.8, 101.1)
- added L1: 6.8uH, Inductor_SMD:L_Vishay_IHLP-2525, F.Cu at (-35.9, 122.0)
- added L2: 6.8uH, Inductor_SMD:L_Vishay_IHLP-2525, F.Cu at (-227.3, 86.7)
- added L3: 6.8uH, Inductor_SMD:L_Vishay_IHLP-2525, F.Cu at (-227.3, 94.7)
- added L4: 6.8uH, Inductor_SMD:L_Vishay_IHLP-2525, F.Cu at (-227.3, 102.6)
- added M1: Fan_4pin, footprints:JST_B4B-PH-SM4-TBT_LF__SN_, F.Cu at (-29.4, 66.0)
- added M2: CSD17571Q2, Package_SON:WSON-6-1EP_2x2mm_P0.65mm_EP1x1.6mm_ThermalVias, F.Cu at (-230.2, 108.4)
- added M3: CSD17571Q2, Package_SON:WSON-6-1EP_2x2mm_P0.65mm_EP1x1.6mm_ThermalVias, F.Cu at (-230.2, 112.1)
- added MOSFET2(Q4)1: SIS412DN-T1-GE3, footprints:POWERPAK_1212-8, F.Cu at (-54.5, 116.5)
- added MOSFET4(Q5)1: SIS412DN-T1-GE3, footprints:POWERPAK_1212-8, F.Cu at (-54.5, 121.5)
- added Q3: SI7135DP-T1-GE3, Package_SO:PowerPAK_SO-8_Single, F.Cu at (-208.7, 99.9)
- added Q4: 2N7002, Package_TO_SOT_SMD:SOT-23, F.Cu at (-101.3, 114.3)
- added Q5: 2SK3018, Package_TO_SOT_SMD:SOT-23, F.Cu at (-101.3, 118.9)
- added Q6: 2SK3018, Package_TO_SOT_SMD:SOT-23, F.Cu at (-101.3, 123.6)
- added Q7: 2SK3018, Package_TO_SOT_SMD:SOT-23, F.Cu at (-101.3, 128.2)
- added Q8: 2N7002, Package_TO_SOT_SMD:SOT-23, F.Cu at (-202.2, 111.8)
- added Q9: SI7135DP-T1-GE3, Package_SO:PowerPAK_SO-8_Single, F.Cu at (-208.7, 106.5)
- added R1: 27.4, Resistor_SMD:R_0402_1005Metric, F.Cu at (-186.0, 38.6)
- added R10: 150, Resistor_SMD:R_0402_1005Metric, F.Cu at (-37.8, 41.9)
- added R100: 2.2K/1%, Resistor_SMD:R_0402_1005Metric, F.Cu at (-91.6, 118.9)
- added R101: 150, Resistor_SMD:R_0402_1005Metric, F.Cu at (-34.9, 41.9)
- added R102: 100, Resistor_SMD:R_0402_1005Metric, F.Cu at (-34.9, 43.9)
- added R103: 150, Resistor_SMD:R_0402_1005Metric, F.Cu at (-34.9, 45.9)
- added R104: 100, Resistor_SMD:R_0402_1005Metric, F.Cu at (-34.9, 47.9)
- added R105: 1.33k, Resistor_SMD:R_0402_1005Metric, F.Cu at (-215.1, 91.7)
- added R106: 1.5k, Resistor_SMD:R_0402_1005Metric, F.Cu at (-91.6, 120.9)
- added R107: 68.1k/10%, Resistor_SMD:R_0402_1005Metric, F.Cu at (-34.7, 105.6)
- added R108: 2.4k, Resistor_SMD:R_0402_1005Metric, F.Cu at (-31.8, 93.7)
- added R109: 1k, Resistor_SMD:R_0402_1005Metric, F.Cu at (-31.8, 95.7)
- added R11: 10k, Resistor_SMD:R_0402_1005Metric, F.Cu at (-31.9, 22.1)
- added R110: 220, Resistor_SMD:R_0402_1005Metric, F.Cu at (-31.8, 97.7)
- added R12: 15R, Resistor_SMD:R_0402_1005Metric, F.Cu at (-31.9, 24.1)
- added R13: 10k±1%, Resistor_SMD:R_0402_1005Metric, F.Cu at (-37.8, 43.9)
- added R14: 2.2k, Resistor_SMD:R_0402_1005Metric, F.Cu at (-220.9, 83.7)
- added R15: 10k, Resistor_SMD:R_0402_1005Metric, F.Cu at (-220.9, 85.7)
- added R16: 100k, Resistor_SMD:R_0402_1005Metric, F.Cu at (-37.8, 45.9)
- added R17: 470, Resistor_SMD:R_0402_1005Metric, F.Cu at (-37.8, 47.9)
- added R18: 1.5k, Resistor_SMD:R_0402_1005Metric, F.Cu at (-220.9, 87.7)
- added R2: 27.4, Resistor_SMD:R_0402_1005Metric, F.Cu at (-186.0, 40.6)
- added R21: 470k, Resistor_SMD:R_0402_1005Metric, F.Cu at (-220.9, 89.7)
- added R22: 10K/1%, Resistor_SMD:R_0402_1005Metric, F.Cu at (-86.0, 0.37)
- added R23: 4.7K/1%, Resistor_SMD:R_0402_1005Metric, F.Cu at (-37.8, 63.7)
- added R24: 21.5K/1%, Resistor_SMD:R_0402_1005Metric, F.Cu at (-37.8, 65.7)
- added R25: 1.5k, Resistor_SMD:R_0402_1005Metric, F.Cu at (-37.8, 67.7)
- added R26: 100R/1%, Resistor_SMD:R_0402_1005Metric, F.Cu at (-37.8, 69.7)
- added R27: 4.7K/1%, Resistor_SMD:R_0402_1005Metric, F.Cu at (-37.8, 71.7)
- added R28: 2.2K/1%, Resistor_SMD:R_0402_1005Metric, F.Cu at (-97.4, 112.9)
- added R29: 10k, Resistor_SMD:R_0402_1005Metric, F.Cu at (-31.9, 26.1)
- added R3: 10k, Resistor_SMD:R_0402_1005Metric, F.Cu at (-186.0, 42.6)
- added R30: 0R, Resistor_SMD:R_0402_1005Metric, F.Cu at (-31.9, 28.1)
- added R31: 9.09k, Resistor_SMD:R_0402_1005Metric, F.Cu at (-40.6, 93.7)
- added R32: 100, Resistor_SMD:R_0402_1005Metric, F.Cu at (-40.6, 95.7)
- added R33: 430, Resistor_SMD:R_0402_1005Metric, F.Cu at (-40.6, 97.7)
- added R34: 43k/10%, Resistor_SMD:R_0402_1005Metric, F.Cu at (-40.6, 99.7)
- added R35: 5.1k/10%, Resistor_SMD:R_0603_1608Metric, F.Cu at (-33.2, 109.1)
- added R36: 34k, Resistor_SMD:R_0402_1005Metric, F.Cu at (-40.6, 101.7)
- added R37: 10k, Resistor_SMD:R_0402_1005Metric, F.Cu at (-40.6, 103.6)
- added R38: 10k, Resistor_SMD:R_0402_1005Metric, F.Cu at (-40.6, 105.6)
- added R39: 10k, Resistor_SMD:R_0402_1005Metric, F.Cu at (-37.6, 93.7)
- added R4: 1k, Resistor_SMD:R_0402_1005Metric, F.Cu at (-186.0, 44.6)
- added R40: 100k, Resistor_SMD:R_0402_1005Metric, F.Cu at (-37.6, 95.7)
- added R41: 1k, Resistor_SMD:R_0402_1005Metric, F.Cu at (-37.6, 97.7)
- added R42: 20k, Resistor_SMD:R_0402_1005Metric, F.Cu at (-37.8, 73.7)
- added R43: 2k, Resistor_SMD:R_0402_1005Metric, F.Cu at (-37.6, 99.7)
- added R44: 10k, Resistor_SMD:R_0402_1005Metric, F.Cu at (-37.6, 101.7)
- added R45: 150, Resistor_SMD:R_0402_1005Metric, F.Cu at (-37.6, 103.6)
- added R46: 560, Resistor_SMD:R_0402_1005Metric, F.Cu at (-37.6, 105.6)
- added R47: 100, Resistor_SMD:R_0402_1005Metric, F.Cu at (-34.7, 93.7)
- added R48: 10, Resistor_SMD:R_0402_1005Metric, F.Cu at (-34.7, 95.7)
- added R49: 100k, Resistor_SMD:R_0402_1005Metric, F.Cu at (-220.9, 91.7)
- added R5: 1k, Resistor_SMD:R_0402_1005Metric, F.Cu at (-186.0, 46.6)
- added R50: 2, Resistor_SMD:R_0402_1005Metric, F.Cu at (-34.7, 97.7)
- added R51: 100k, Resistor_SMD:R_0402_1005Metric, F.Cu at (-34.7, 99.7)
- added R52: 1k, Resistor_SMD:R_0402_1005Metric, F.Cu at (-34.7, 101.7)
- added R53: 150, Resistor_SMD:R_0402_1005Metric, F.Cu at (-220.9, 93.7)
- added R54: 100k, Resistor_SMD:R_0402_1005Metric, F.Cu at (-220.9, 95.7)
- added R55: 8.2k, Capacitor_SMD:C_0402_1005Metric, F.Cu at (-198.4, 87.7)
- added R56: 100k, Resistor_SMD:R_0402_1005Metric, F.Cu at (-218.0, 83.7)
- added R57: 22k, Resistor_SMD:R_0402_1005Metric, F.Cu at (-218.0, 85.7)
- added R58: 100R/1%, Resistor_SMD:R_0402_1005Metric, F.Cu at (-218.0, 87.7)
- added R59: 10K/1%, Resistor_SMD:R_0402_1005Metric, F.Cu at (-218.0, 89.7)
- added R6: 0, Resistor_SMD:R_1206_3216Metric, F.Cu at (-174.2, 51.0)
- added R60: 100R/1%, Resistor_SMD:R_0402_1005Metric, F.Cu at (-218.0, 91.7)
- added R61: 10K/1%, Resistor_SMD:R_0402_1005Metric, F.Cu at (-218.0, 93.7)
- added R62: 1K/1%, Resistor_SMD:R_0402_1005Metric, F.Cu at (-218.0, 95.7)
- added R63: 10K/1%, Resistor_SMD:R_0402_1005Metric, F.Cu at (-215.1, 83.7)
- added R64: 2.2K/1%, Resistor_SMD:R_0402_1005Metric, F.Cu at (-215.1, 85.7)
- added R65: 68k, Resistor_SMD:R_0402_1005Metric, F.Cu at (-34.7, 103.6)
- added R66: 100k, Resistor_SMD:R_0402_1005Metric, F.Cu at (-37.8, 49.9)
- added R67: 2k, Resistor_SMD:R_0402_1005Metric, F.Cu at (-215.1, 87.7)
- added R68: 100, Resistor_SMD:R_0402_1005Metric, F.Cu at (-215.1, 89.7)
- added R69: 10K/1%, Resistor_SMD:R_0402_1005Metric, F.Cu at (-148.1, 100.9)
- added R7: 1K/1%, Resistor_SMD:R_0402_1005Metric, F.Cu at (-86.0, -1.62)
- added R70: 1K/1%, Resistor_SMD:R_0402_1005Metric, F.Cu at (-148.1, 102.9)
- added R71: 120K/1%, Resistor_SMD:R_0402_1005Metric, F.Cu at (-148.1, 104.9)
- added R72: 0R/1%, Resistor_SMD:R_0402_1005Metric, F.Cu at (-190.7, 124.1)
- added R73: 0R/1%, Resistor_SMD:R_0402_1005Metric, F.Cu at (-190.7, 126.0)
- added R74: 10K/1%, Resistor_SMD:R_0402_1005Metric, F.Cu at (-190.7, 128.0)
- added R75: 10K/1%, Resistor_SMD:R_0402_1005Metric, F.Cu at (-190.7, 130.0)
- added R76: 100K/1%, Resistor_SMD:R_0402_1005Metric, F.Cu at (-86.0, 2.36)
- added R77: 100K/1%, Resistor_SMD:R_0402_1005Metric, F.Cu at (-86.0, 4.35)
- added R78: 0R, Resistor_SMD:R_0402_1005Metric, F.Cu at (-31.9, 30.1)
- added R79: 0R, Resistor_SMD:R_0402_1005Metric, F.Cu at (-29.0, 22.1)
- added R8: 453k, Resistor_SMD:R_0402_1005Metric, F.Cu at (-37.8, 37.9)
- added R80: 1M/1%, Resistor_SMD:R_0402_1005Metric, F.Cu at (-97.4, 114.9)
- added R81: 15R, Resistor_SMD:R_0402_1005Metric, F.Cu at (-29.0, 24.1)
- added R82: 15R, Resistor_SMD:R_0402_1005Metric, F.Cu at (-29.0, 26.1)
- added R83: 0R, Resistor_SMD:R_0402_1005Metric, F.Cu at (-29.0, 28.1)
- added R84: 0R, Resistor_SMD:R_0402_1005Metric, F.Cu at (-29.0, 30.1)
- added R85: 1k/5%, Resistor_SMD:R_0402_1005Metric, F.Cu at (-34.9, 37.9)
- added R86: 2.2K/1%, Resistor_SMD:R_0402_1005Metric, F.Cu at (-97.4, 116.9)
- added R87: 20k, Resistor_SMD:R_0402_1005Metric, F.Cu at (-97.4, 118.9)
- added R88: 470R/1%, Resistor_SMD:R_0402_1005Metric, F.Cu at (-97.4, 120.9)
- added R89: 470R/1%, Resistor_SMD:R_0402_1005Metric, F.Cu at (-97.4, 122.9)
- added R9: 150, Resistor_SMD:R_0402_1005Metric, F.Cu at (-37.8, 39.9)
- added R90: 470R/1%, Resistor_SMD:R_0402_1005Metric, F.Cu at (-94.5, 112.9)
- added R91: 470R/1%, Resistor_SMD:R_0402_1005Metric, F.Cu at (-94.5, 114.9)
- added R92: 1K/1%, Resistor_SMD:R_0402_1005Metric, F.Cu at (-94.5, 116.9)
- added R93: 470R/1%, Resistor_SMD:R_0402_1005Metric, F.Cu at (-94.5, 118.9)
- added R94: 150, Resistor_SMD:R_0402_1005Metric, F.Cu at (-34.9, 39.9)
- added R95: 470R/1%, Resistor_SMD:R_0402_1005Metric, F.Cu at (-94.5, 120.9)
- added R96: 2.2K/1%, Resistor_SMD:R_0402_1005Metric, F.Cu at (-94.5, 122.9)
- added R97: 470R/1%, Resistor_SMD:R_0402_1005Metric, F.Cu at (-91.6, 112.9)
- added R98: 470R/1%, Resistor_SMD:R_0402_1005Metric, F.Cu at (-91.6, 114.9)
- added R99: 2.2K/1%, Resistor_SMD:R_0402_1005Metric, F.Cu at (-91.6, 116.9)
- added R_{AC}1: 0.01, footprints:RESC_WSHM2818R0150FEA, F.Cu at (-52.6, 96.2)
- added R_{AC}2: 0.01, footprints:RESC_WSHM2818R0150FEA, F.Cu at (-52.6, 103.3)
- added R_{CHG}1: 220/5%, Resistor_SMD:R_0402_1005Metric, F.Cu at (-34.9, 49.9)
- added R_{DSG}1: 470/5%, Resistor_SMD:R_0402_1005Metric, F.Cu at (-32.0, 37.9)
- added R_{GS}1: 4.7M, Resistor_SMD:R_0402_1005Metric, F.Cu at (-32.0, 39.9)
- added R_{GS}2: 4.7M, Resistor_SMD:R_0402_1005Metric, F.Cu at (-32.0, 41.9)
- added R_{SNS}1: 4m, Resistor_SMD:R_0402_1005Metric, F.Cu at (-32.0, 43.9)
- added R_{SR}1: 0.01/1%, footprints:RESC_WSHM2818R0150FEA, F.Cu at (-52.6, 110.4)
- added Rcomp2: 200, Resistor_SMD:R_0402_1005Metric, F.Cu at (-215.1, 93.7)
- added Rcomp3: 27, Resistor_SMD:R_0402_1005Metric, F.Cu at (-215.1, 95.7)
- added Rcomp4: 10, Resistor_SMD:R_0402_1005Metric, F.Cu at (-212.2, 83.7)
- added Rfbb1: 604, Resistor_SMD:R_0402_1005Metric, F.Cu at (-212.2, 85.7)
- added Rfbb2: 30, Resistor_SMD:R_0402_1005Metric, F.Cu at (-212.2, 87.7)
- added Rfbt1: 10k, Resistor_SMD:R_0402_1005Metric, F.Cu at (-212.2, 89.7)
- added S1: Keyswitch, footprints:SW_PG151101S11, F.Cu at (-223.0, -77.2)
- added S10: Keyswitch, footprints:SW_PG151101S11, F.Cu at (-223.0, -10.3)
- added S100: Keyswitch, footprints:SW_PG151101S11, F.Cu at (-114.5, -10.3)
- added S101: Keyswitch, footprints:SW_PG151101S11, F.Cu at (-114.5, -2.85)
- added S102: Keyswitch, footprints:SW_PG151101S11, F.Cu at (-114.5, 4.59)
- added S103: Keyswitch, footprints:SW_PG151101S11, F.Cu at (-114.5, 12.0)
- added S104: Keyswitch, footprints:SW_PG151101S11, F.Cu at (-114.5, 19.5)
- added S11: Keyswitch, footprints:SW_PG151101S11, F.Cu at (-223.0, -2.85)
- added S12: Keyswitch, footprints:SW_PG151101S11, F.Cu at (-223.0, 4.59)
- added S13: Keyswitch, footprints:SW_PG151101S11, F.Cu at (-223.0, 12.0)
- added S14: Keyswitch, footprints:SW_PG151101S11, F.Cu at (-223.0, 19.5)
- added S15: Keyswitch, footprints:SW_PG151101S11, F.Cu at (-223.0, 26.9)
- added S16: Keyswitch, footprints:SW_PG151101S11, F.Cu at (-204.9, -77.2)
- added S17: Keyswitch, footprints:SW_PG151101S11, F.Cu at (-204.9, -69.8)
- added S18: Keyswitch, footprints:SW_PG151101S11, F.Cu at (-204.9, -62.4)
- added S19: Keyswitch, footprints:SW_PG151101S11, F.Cu at (-204.9, -54.9)
- added S2: Keyswitch, footprints:SW_PG151101S11, F.Cu at (-223.0, -69.8)
- added S20: Keyswitch, footprints:SW_PG151101S11, F.Cu at (-204.9, -47.5)
- added S21: Keyswitch, footprints:SW_PG151101S11, F.Cu at (-204.9, -40.0)
- added S22: Keyswitch, footprints:SW_PG151101S11, F.Cu at (-204.9, -32.6)
- added S23: Keyswitch, footprints:SW_PG151101S11, F.Cu at (-204.9, -25.2)
- added S24: Keyswitch, footprints:SW_PG151101S11, F.Cu at (-204.9, -17.7)
- added S25: Keyswitch, footprints:SW_PG151101S11, F.Cu at (-204.9, -10.3)
- added S26: Keyswitch, footprints:SW_PG151101S11, F.Cu at (-204.9, -2.85)
- added S27: Keyswitch, footprints:SW_PG151101S11, F.Cu at (-204.9, 4.59)
- added S28: Keyswitch, footprints:SW_PG151101S11, F.Cu at (-204.9, 12.0)
- added S29: Keyswitch, footprints:SW_PG151101S11, F.Cu at (-204.9, 19.5)
- added S3: Keyswitch, footprints:SW_PG151101S11, F.Cu at (-223.0, -62.4)
- added S30: Keyswitch, footprints:SW_PG151101S11, F.Cu at (-204.9, 26.9)
- added S31: Keyswitch, footprints:SW_PG151101S11, F.Cu at (-186.8, -77.2)
- added S32: Keyswitch, footprints:SW_PG151101S11, F.Cu at (-186.8, -69.8)
- added S33: Keyswitch, footprints:SW_PG151101S11, F.Cu at (-186.8, -62.4)
- added S34: Keyswitch, footprints:SW_PG151101S11, F.Cu at (-186.8, -54.9)
- added S35: Keyswitch, footprints:SW_PG151101S11, F.Cu at (-186.8, -47.5)
- added S36: Keyswitch, footprints:SW_PG151101S11, F.Cu at (-186.8, -40.0)
- added S37: Keyswitch, footprints:SW_PG151101S11, F.Cu at (-186.8, -32.6)
- added S38: Keyswitch, footprints:SW_PG151101S11, F.Cu at (-186.8, -25.2)
- added S39: Keyswitch, footprints:SW_PG151101S11, F.Cu at (-186.8, -17.7)
- added S4: Keyswitch, footprints:SW_PG151101S11, F.Cu at (-223.0, -54.9)
- added S40: Keyswitch, footprints:SW_PG151101S11, F.Cu at (-186.8, -10.3)
- added S41: Keyswitch, footprints:SW_PG151101S11, F.Cu at (-186.8, -2.85)
- added S42: Keyswitch, footprints:SW_PG151101S11, F.Cu at (-186.8, 4.59)
- added S43: Keyswitch, footprints:SW_PG151101S11, F.Cu at (-186.8, 12.0)
- added S44: Keyswitch, footprints:SW_PG151101S11, F.Cu at (-186.8, 19.5)
- added S45: Keyswitch, footprints:SW_PG151101S11, F.Cu at (-186.8, 26.9)
- added S46: Keyswitch, footprints:SW_PG151101S11, F.Cu at (-168.7, -77.2)
- added S47: Keyswitch, footprints:SW_PG151101S11, F.Cu at (-168.7, -69.8)
- added S48: Keyswitch, footprints:SW_PG151101S11, F.Cu at (-168.7, -62.4)
- added S49: Keyswitch, footprints:SW_PG151101S11, F.Cu at (-168.7, -54.9)
- added S5: Keyswitch, footprints:SW_PG151101S11, F.Cu at (-223.0, -47.5)
- added S50: Keyswitch, footprints:SW_PG151101S11, F.Cu at (-168.7, -47.5)
- added S51: Keyswitch, footprints:SW_PG151101S11, F.Cu at (-168.7, -40.0)
- added S52: Keyswitch, footprints:SW_PG151101S11, F.Cu at (-168.7, -32.6)
- added S53: Keyswitch, footprints:SW_PG151101S11, F.Cu at (-168.7, -25.2)
- added S54: Keyswitch, footprints:SW_PG151101S11, F.Cu at (-168.7, -17.7)
- added S55: Keyswitch, footprints:SW_PG151101S11, F.Cu at (-168.7, -10.3)
- added S56: Keyswitch, footprints:SW_PG151101S11, F.Cu at (-168.7, -2.85)
- added S57: Keyswitch, footprints:SW_PG151101S11, F.Cu at (-168.7, 4.59)
- added S58: Keyswitch, footprints:SW_PG151101S11, F.Cu at (-168.7, 12.0)
- added S59: Keyswitch, footprints:SW_PG151101S11, F.Cu at (-168.7, 19.5)
- added S6: Keyswitch, footprints:SW_PG151101S11, F.Cu at (-223.0, -40.0)
- added S60: Keyswitch, footprints:SW_PG151101S11, F.Cu at (-168.7, 26.9)
- added S61: Keyswitch, footprints:SW_PG151101S11, F.Cu at (-150.7, -77.2)
- added S62: Keyswitch, footprints:SW_PG151101S11, F.Cu at (-150.7, -69.8)
- added S63: Keyswitch, footprints:SW_PG151101S11, F.Cu at (-150.7, -62.4)
- added S64: Keyswitch, footprints:SW_PG151101S11, F.Cu at (-150.7, -54.9)
- added S65: Keyswitch, footprints:SW_PG151101S11, F.Cu at (-150.7, -47.5)
- added S66: Keyswitch, footprints:SW_PG151101S11, F.Cu at (-150.7, -40.0)
- added S67: Keyswitch, footprints:SW_PG151101S11, F.Cu at (-150.7, -32.6)
- added S68: Keyswitch, footprints:SW_PG151101S11, F.Cu at (-150.7, -25.2)
- added S69: Keyswitch, footprints:SW_PG151101S11, F.Cu at (-150.7, -17.7)
- added S7: Keyswitch, footprints:SW_PG151101S11, F.Cu at (-223.0, -32.6)
- added S70: Keyswitch, footprints:SW_PG151101S11, F.Cu at (-150.7, -10.3)
- added S71: Keyswitch, footprints:SW_PG151101S11, F.Cu at (-150.7, -2.85)
- added S72: Keyswitch, footprints:SW_PG151101S11, F.Cu at (-150.7, 4.59)
- added S73: Keyswitch, footprints:SW_PG151101S11, F.Cu at (-150.7, 12.0)
- added S74: Keyswitch, footprints:SW_PG151101S11, F.Cu at (-150.7, 19.5)
- added S75: Keyswitch, footprints:SW_PG151101S11, F.Cu at (-150.7, 26.9)
- added S76: Keyswitch, footprints:SW_PG151101S11, F.Cu at (-132.6, -77.2)
- added S77: Keyswitch, footprints:SW_PG151101S11, F.Cu at (-132.6, -69.8)
- added S78: Keyswitch, footprints:SW_PG151101S11, F.Cu at (-132.6, -62.4)
- added S79: Keyswitch, footprints:SW_PG151101S11, F.Cu at (-132.6, -54.9)
- added S8: Keyswitch, footprints:SW_PG151101S11, F.Cu at (-223.0, -25.2)
- added S80: Keyswitch, footprints:SW_PG151101S11, F.Cu at (-132.6, -47.5)
- added S81: Keyswitch, footprints:SW_PG151101S11, F.Cu at (-132.6, -40.0)
- added S82: Keyswitch, footprints:SW_PG151101S11, F.Cu at (-132.6, -32.6)
- added S83: Keyswitch, footprints:SW_PG151101S11, F.Cu at (-132.6, -25.2)
- added S84: Keyswitch, footprints:SW_PG151101S11, F.Cu at (-132.6, -17.7)
- added S85: Keyswitch, footprints:SW_PG151101S11, F.Cu at (-132.6, -10.3)
- added S86: Keyswitch, footprints:SW_PG151101S11, F.Cu at (-132.6, -2.85)
- added S87: Keyswitch, footprints:SW_PG151101S11, F.Cu at (-132.6, 4.59)
- added S88: Keyswitch, footprints:SW_PG151101S11, F.Cu at (-132.6, 12.0)
- added S89: Keyswitch, footprints:SW_PG151101S11, F.Cu at (-132.6, 19.5)
- added S9: Keyswitch, footprints:SW_PG151101S11, F.Cu at (-223.0, -17.7)
- added S90: Keyswitch, footprints:SW_PG151101S11, F.Cu at (-132.6, 26.9)
- added S91: Keyswitch, footprints:SW_PG151101S11, F.Cu at (-114.5, -77.2)
- added S92: Keyswitch, footprints:SW_PG151101S11, F.Cu at (-114.5, -69.8)
- added S93: Keyswitch, footprints:SW_PG151101S11, F.Cu at (-114.5, -62.4)
- added S94: Keyswitch, footprints:SW_PG151101S11, F.Cu at (-114.5, -54.9)
- added S95: Keyswitch, footprints:SW_PG151101S11, F.Cu at (-114.5, -47.5)
- added S96: Keyswitch, footprints:SW_PG151101S11, F.Cu at (-114.5, -40.0)
- added S97: Keyswitch, footprints:SW_PG151101S11, F.Cu at (-114.5, -32.6)
- added S98: Keyswitch, footprints:SW_PG151101S11, F.Cu at (-114.5, -25.2)
- added S99: Keyswitch, footprints:SW_PG151101S11, F.Cu at (-114.5, -17.7)
- added SW1: SW_Push, footprints:SW_TS-1187A-B-A-B, F.Cu at (-217.5, 100.0)
- added SW2: SW_Push, footprints:SW_TS-1187A-B-A-B, F.Cu at (-217.5, 106.6)
- added SW_{HibernateBattery}1: CFS-0102TA, footprints:SW_CFS-0102MA_NDC-L, F.Cu at (-24.8, 55.9)
- added TH2: 103AT, Resistor_SMD:R_0603_1608Metric, F.Cu at (-33.2, 111.7)
- added TH_103AT_1: 10k@25°C, Resistor_SMD:R_0201_0603Metric, F.Cu at (-20.2, 50.4)
- added TP1: TestPoint_Small, TestPoint:TestPoint_Pad_D1.0mm, F.Cu at (-175.5, 32.2)
- added TP10: TestPoint, TestPoint:TestPoint_Pad_D1.0mm, F.Cu at (-80.0, -13.0)
- added TP11: TestPoint, TestPoint:TestPoint_Pad_D1.0mm, F.Cu at (-34.9, 73.9)
- added TP12: TestPoint, TestPoint:TestPoint_Pad_D1.0mm, F.Cu at (-34.9, 76.9)
- added TP13: KB_USB_D-, TestPoint:TestPoint_Loop_D1.80mm_Drill1.0mm_Beaded, F.Cu at (-185.2, 69.4)
- added TP14: TestPoint, TestPoint:TestPoint_Pad_1.0x1.0mm, F.Cu at (-34.9, 22.7)
- added TP15: TestPoint, TestPoint:TestPoint_Pad_1.0x1.0mm, F.Cu at (-34.9, 25.7)
- added TP16: TestPoint, TestPoint:TestPoint_Pad_1.0x1.0mm, F.Cu at (-34.9, 28.8)
- added TP17: KB_USB_D+, TestPoint:TestPoint_Loop_D1.80mm_Drill1.0mm_Beaded, F.Cu at (-185.2, 74.0)
- added TP18: TestPoint, TestPoint:TestPoint_Pad_1.0x1.0mm, F.Cu at (-34.9, 31.8)
- added TP2: TestPoint_Small, TestPoint:TestPoint_Pad_D1.0mm, F.Cu at (-175.5, 35.2)
- added TP3: TestPoint_Small, TestPoint:TestPoint_Pad_D1.0mm, F.Cu at (-175.5, 38.3)
- added TP4: TestPoint_Small, TestPoint:TestPoint_Pad_D1.0mm, F.Cu at (-172.4, 32.2)
- added TP5: TestPoint_Small, TestPoint:TestPoint_Pad_D1.0mm, F.Cu at (-172.4, 35.2)
- added TP6: TestPoint_Small, TestPoint:TestPoint_Pad_D1.0mm, F.Cu at (-172.4, 38.3)
- added TP7: TestPoint_Small, TestPoint:TestPoint_Pad_D1.0mm, F.Cu at (-169.4, 32.2)
- added TP8: TestPoint_Small, TestPoint:TestPoint_Pad_D1.0mm, F.Cu at (-169.4, 35.2)
- added TP9: TestPoint_Small, TestPoint:TestPoint_Pad_D1.0mm, F.Cu at (-169.4, 38.3)
- added U1: W25Q128JVS, footprints:SOIC_128JVSIQ_WIN, F.Cu at (-182.3, 34.1)
- added U10: CH224K, footprints:ESSOP-10_L4.9-W3.9-P1.0-LS6.0-TL-EP, F.Cu at (-152.6, 104.2)
- added U11: CSD85302L, footprints:YME0004A-MFG, F.Cu at (-19.5, 48.0)
- added U12: LTC4412ES6#TRMPBF, Package_TO_SOT_SMD:TSOT-23-6, F.Cu at (-208.2, 94.4)
- added U13: SP3004-04XTG, Package_TO_SOT_SMD:SOT-563, F.Cu at (-85.2, 113.4)
- added U14: SP3004-04XTG, Package_TO_SOT_SMD:SOT-563, F.Cu at (-85.2, 116.4)
- added U2: SC091413, footprints:QFN56_7X7_RPI, F.Cu at (-182.7, 62.2)
- added U3: BQ7791500PWR, footprints:PW24_TEX, F.Cu at (-25.9, 41.7)
- added U4: BQ34Z100PWR-R2, footprints:PW14_TEX, F.Cu at (-26.1, 49.9)
- added U5: TPS54302, Package_TO_SOT_SMD:SOT-23-6, F.Cu at (-208.2, 85.1)
- added U6: BQ24617RGER, footprints:RGE24_2P45X2P45, F.Cu at (-44.7, 122.5)
- added U7: TPS40345DRCR, footprints:DRC0010J, F.Cu at (-211.0, 112.0)
- added U8: TPS54302, Package_TO_SOT_SMD:SOT-23-6, F.Cu at (-208.2, 89.8)
- added U9: CDDFN10-0524P, Package_DFN_QFN:Diodes_UDFN-10_1.0x2.5mm_P0.5mm, F.Cu at (-188.9, 106.0)
- added X1: ABM8-272-T3, footprints:ABM8-272-T3_ABR, F.Cu at (-173.2, 46.7)
Other:
- board outline added: 49.6 x 53.5 mm
