File: KiCad/RDAT/RDAT.kicad_pcb (KiCad board)
At the start: 2 copper layers, 49.6 x 53.5 mm, 530 parts, among them J1 Conn_01x02, J16 MDT420E03001, J18 MUSBRM1C130, J2 Conn_01x02, J3 Conn_01x02, J4 Bus_M.2_Socket_B, J5 USB_A_Stacked, J6 HDMI_A, M1 Fan_4pin, M2 CSD17571Q2, M3 CSD17571Q2, Q3 SI7135DP-T1-GE3, Q4 2N7002, Q5 2SK3018, Q6 2SK3018, Q7 2SK3018, Q8 2N7002, Q9 SI7135DP-T1-GE3, SW1 SW_Push, SW2 SW_Push, U1 W25Q128JVS, U10 CH224K, U11 CSD85302L, U12 LTC4412ES6#TRMPBF, U13 SP3004-04XTG, U14 SP3004-04XTG, U2 SC091413, U3 BQ7791500PWR, U4 BQ34Z100PWR-R2, U5 TPS54302, U6 BQ24617RGER, U7 TPS40345DRCR, U8 TPS54302, U9 CDDFN10-0524P, X1 ABM8-272-T3

Commit message: Updated Layout
Parts:
- S1, S10, S100, S101, S102, S103, S104, S11, S12, S13, S14, S15, S16, S17, S18, S19, S2, S20, S21, S22, S23, S24, S25, S26, S27, S28, S29, S3, S30, S31, S32, S33, S34, S35, S36, S37, S38, S39, S4, S40, S41, S42, S43, S44, S45, S46, S47, S48, S49, S5, S50, S51, S52, S53, S54, S55, S56, S57, S58, S59, S6, S60, S61, S62, S63, S64, S65, S66, S67, S68, S69, S7, S70, S71, S72, S73, S74, S75, S76, S77, S78, S79, S8, S80, S81, S82, S83, S84, S85, S86, S87, S88, S89, S9, S90, S91, S92, S93, S94, S95, S96, S97, S98, S99: moved to B.Cu
- moved S65 578.8 mm to (420.8, -139.0)
- moved S64 562.6 mm to (405.6, -139.0)
- moved S78 556.1 mm to (420.9, -116.9)
- moved S90 552.8 mm to (405.7, -98.8)
- moved S59 550.1 mm to (374.3, 107.5)
- moved S63 546.5 mm to (390.5, -139.0)
- moved S75 545.3 mm to (375.3, -116.9)
- moved S104 544.9 mm to (421.1, -80.8)
- moved S77 540.3 mm to (405.7, -116.9)
- moved S60 539.8 mm to (344.9, -139.0)
- moved S89 536.3 mm to (390.5, -98.8)
- moved S91 535.8 mm to (420.9, -98.8)
- moved S52 530.7 mm to (348.1, 87.7)
- moved S13 530.5 mm to (307.3, 30.7)
- moved S62 530.5 mm to (375.3, -139.0)
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
Commit message: Placed a lot of components
Parts:
- removed C68: 100fP/50v, Capacitor_SMD:C_0402_1005Metric
- removed D104: Diode, Diode_SMD:D_MiniMELF
- removed J3: Conn_01x02, Connector_PinHeader_1.00mm:PinHeader_1x02_P1.00mm_Vertical
- removed SW1, SW2: SW_Push, footprints:SW_TS-1187A-B-A-B
- added C73: 100fP/50v, Capacitor_SMD:C_0402_1005Metric, F.Cu at (625.7, 229.6)
- added J7: SF72S006VBDR2500, Connector_JAE:JAE_SIM_Card_SF72S006, F.Cu at (617.8, 225.3)
- added S105: TS-1187A-B-A-B, footprints:SW_TS-1187A-B-A-B, F.Cu at (418.6, 327.3)
- S104: value Keyswitch -> TS-1187A-B-A-B; footprint footprints:SW_PG151101S11 -> footprints:SW_TS-1187A-B-A-B; moved to F.Cu
- moved C80 905.0 mm to (702.6, 238.5), turned to 180 degrees
- moved C81 904.8 mm to (702.6, 239.5), turned to 180 degrees
- moved R72 901.2 mm to (702.6, 243.0)
- moved C84 893.7 mm to (691.0, 247.8)
- moved C85 893.5 mm to (691.0, 248.7)
- moved C82 892.0 mm to (691.0, 231.2)
- moved C83 891.6 mm to (691.0, 230.2)
- moved R74 889.3 mm to (691.0, 244.5), turned to 180 degrees
- moved R73 889.3 mm to (691.0, 242.1), turned to 180 degrees
- moved R75 889.0 mm to (691.0, 243.5)
- moved J16 883.9 mm to (695.3, 239.5), turned to -90 degrees
- moved R60 777.4 mm to (552.6, 194.0), turned to 90 degrees
- moved R58 777.0 mm to (551.6, 194.0), turned to 90 degrees
- moved D63 775.1 mm to (503.8, 356.2), turned to 90 degrees
- moved D62 762.9 mm to (484.6, 365.1), turned to 90 degrees
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Connections:
- D128 pad 1: /usbC_Switcher/CC2 -> /usbC_Switcher/CC1
- J1 pad 1: /Keyboard/~{USB_BOOT} -> GND
- J1 pad 2: GND -> /Keyboard/~{USB_BOOT}
- J18 pad A10: (no net) -> unconnected-(J18-RX2--PadA10)
- J18 pad A11: (no net) -> unconnected-(J18-RX2+-PadA11)
- J18 pad A2: (no net) -> unconnected-(J18-TX1+-PadA2)
- J18 pad A3: (no net) -> unconnected-(J18-TX1--PadA3)
- J18 pad B10: (no net) -> unconnected-(J18-RX1--PadB10)
- J18 pad B11: (no net) -> unconnected-(J18-RX1+-PadB11)
- J18 pad B2: (no net) -> unconnected-(J18-TX2+-PadB2)
- J18 pad B3: (no net) -> unconnected-(J18-TX2--PadB3)
- J18 pad B5: /usbC_Switcher/CC2 -> unconnected-(J18-VCONN-PadB5)
- J18 pad B6: /usbC_Switcher/PWR_C_D+ -> (no net)
- J18 pad B7: /usbC_Switcher/PWR_C_D- -> (no net)
- M2 pad 1: Net-(M3-S) -> unconnected-(M2-D-Pad1)
- M2 pad 2: Net-(M3-S) -> unconnected-(M2-D-Pad2)
- M2 pad 5: unconnected-(M2-D-Pad5) -> Net-(M3-S)
- M2 pad 6: unconnected-(M2-D-Pad6) -> Net-(M3-S)
- S13 pad 1: /Keyboard/Col_12 -> Net-(S13-Pad1)
- S26 pad 1: /Keyboard/Col_12 -> Net-(S13-Pad1)
- S39 pad 1: /Keyboard/Col_12 -> Net-(S13-Pad1)
- S52 pad 1: /Keyboard/Col_12 -> Net-(S13-Pad1)
- S65 pad 1: /Keyboard/Col_12 -> Net-(S13-Pad1)
- S78 pad 1: /Keyboard/Col_12 -> Net-(S13-Pad1)
- S91 pad 1: /Keyboard/Col_12 -> Net-(S13-Pad1)
- TP13 pad 1: /Keyboard/USB_DM -> /Keyboard/KB_USB_D-
- TP17 pad 1: /Keyboard/USB_DP -> /Keyboard/KB_USB_D+
- U10 pad 6: /usbC_Switcher/CC2 -> /usbC_Switcher/CC1
Routing:
- net /Charging IC/PH: track 0.00 -> 10.1 mm
- net /Charging IC/HIDRV: track 0.00 -> 9.27 mm
- net /Charging IC/LODRV: track 0.00 -> 9.08 mm
Other:
- copper layers 2 -> 4
