File: KiCad/RDAT/RDAT.kicad_pcb (KiCad board)
At the start: 4 copper layers, 49.6 x 53.5 mm, 528 parts, among them J1 Conn_01x02, J16 MDT420E03001, J18 MUSBRM1C130, J2 Conn_01x02, J4 Bus_M.2_Socket_B, J5 USB_A_Stacked, J6 HDMI_A, J7 SF72S006VBDR2500, M1 Fan_4pin, M2 CSD17571Q2, M3 CSD17571Q2, Q3 SI7135DP-T1-GE3, Q4 2N7002, Q5 2SK3018, Q6 2SK3018, Q7 2SK3018, Q8 2N7002, Q9 SI7135DP-T1-GE3, U1 W25Q128JVS, U10 CH224K, U11 CSD85302L, U12 LTC4412ES6#TRMPBF, U13 SP3004-04XTG, U14 SP3004-04XTG, U2 SC091413, U3 BQ7791500PWR, U4 BQ34Z100PWR-R2, U5 TPS54302, U6 BQ24617RGER, U7 TPS40345DRCR, U8 TPS54302, U9 CDDFN10-0524P, X1 ABM8-272-T3

Commit message: added Trace width table
Parts:
- added REF**: Screen Width, footprints:Screen Width, F.Cu at (111.5, 61.5)
- moved R23 354.8 mm to (535.1, 131.0)
- moved R24 354.8 mm to (535.1, 133.0)
- moved R25 354.8 mm to (535.1, 134.9)
- moved R26 354.8 mm to (535.1, 136.9)
- moved R27 354.8 mm to (535.1, 138.9)
- moved R42 354.8 mm to (535.1, 140.9)
- moved D109 354.8 mm to (541.7, 141.1)
- moved M1 354.8 mm to (543.5, 133.2)
- moved C24 354.8 mm to (541.0, 143.5)
- moved TP11 354.8 mm to (538.0, 141.1)
- moved TP12 354.8 mm to (538.0, 144.2)
- moved R86 132.4 mm to (103.5, 194.5)
- moved C27 131.8 mm to (106.0, 210.5)
- moved Q7 122.3 mm to (108.8, 201.6)
- moved Q5 121.4 mm to (109.6, 192.0)
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
Commit message: End Of day commit
Parts:
- removed BT17: 3v, footprints:HARWIN_S8411-45R
- removed J18: MUSBRM1C130, footprints:AMPHENOL_MUSBRM1C130
- removed Q3: SI7135DP-T1-GE3, Package_SO:PowerPAK_SO-8_Single
- removed REF**: Screen Width, footprints:Screen Width
- removed U10: CH224K, footprints:ESSOP-10_L4.9-W3.9-P1.0-LS6.0-TL-EP
- removed U13, U14: SP3004-04XTG, Package_TO_SOT_SMD:SOT-563
- added D104: PESD2USB3UV-TR, Package_TO_SOT_SMD:SOT-23, F.Cu at (73.0, 225.6)
- added D107: PESD2USB3UV-TR, Package_TO_SOT_SMD:SOT-23, F.Cu at (69.8, 229.2)
- added D108: PESD2USB3UV-TR, Package_TO_SOT_SMD:SOT-23, F.Cu at (66.4, 222.0)
- added D115: PESD2USB3UV-TR, Package_TO_SOT_SMD:SOT-23, F.Cu at (66.3, 229.2)
- added J3: S8411-45R, footprints:HARWIN_S8411-45R, F.Cu at (188.3, 197.1)
- added J8: MUSBRM1C130, footprints:AMPHENOL_MUSBRM1C130, F.Cu at (60.0, 193.2)
- added Q10: SI7135DP-T1-GE3, Package_SO:PowerPAK_SO-8_Single, F.Cu at (365.7, 187.6)
- added U15: CH224K, Package_SO:SSOP-10-1EP_3.9x4.9mm_P1mm_EP2.1x3.3mm, F.Cu at (66.4, 190.8)
- A1: footprint footprints:LattePanda_Module_H4.0mm_Horizontal -> footprints:LattePanda_Module_H8.0mm_Horizontal
- D1, D10, D100, D101, D102, D103, D11, D12, D13, D14, D15, D16, D17, D18, D19, D2, D20, D21, D22, D23, D24, D25, D26, D27, D28, D29, D3, D30, D31, D32, D33, D34, D35, D36, D37, D38, D39, D4, D40, D41, D42, D43, D44, D45, D46, D47, D48, D49, D5, D50, D51, D52, D53, D54, D55, D56, D57, D58, D59, D6, D60, D61, D62, D63, D64, D65, D66, D67, D68, D69, D7, D70, D71, D72, D73, D74, D75, D76, D77, D78, D79, D8, D80, D81, D82, D83, D84, D85, D86, D87, D88, D89, D9, D90, D91, D92, D93, D94, D95, D96, D97, D98, D99: footprint Diode_SMD:D_MiniMELF -> Diode_SMD:D_SOD-882; moved to B.Cu
- J7: footprint Connector_JAE:JAE_SIM_Card_SF72S006 -> footprints:SF72S006VBDR2500_JAE
- M2, M3: footprint Package_SON:WSON-6-1EP_2x2mm_P0.65mm_EP1x1.6mm_ThermalVias -> footprints:DQK0006C
- R71: value 120K/1% -> 200k/1%
- U6: footprint footprints:RGE24_2P45X2P45 -> Package_DFN_QFN:Texas_RGE0024H_VQFN-24-1EP_4x4mm_P0.5mm_EP2.7x2.7mm_ThermalVias
- moved H6 450.9 mm to (191.7, 247.7)
- moved R7 438.2 mm to (197.9, 188.9), turned to 180 degrees
- moved TP7 434.5 mm to (11.8, 1.02), turned to 0 degrees
- moved TP8 433.6 mm to (11.8, 4.08), turned to 0 degrees
- moved TP9 432.8 mm to (11.8, 7.12), turned to 0 degrees
- moved TP4 431.2 mm to (8.72, 1.02), turned to 0 degrees
- moved TP5 430.4 mm to (8.72, 4.08), turned to 0 degrees
- moved TP6 429.5 mm to (8.72, 7.12), turned to 0 degrees
- moved TP1 428.0 mm to (5.67, 1.02), turned to 0 degrees
- moved TP2 427.2 mm to (5.67, 4.08), turned to 0 degrees
- moved TP3 426.3 mm to (5.67, 7.12), turned to 0 degrees
- moved R76 413.8 mm to (222.2, 186.3), turned to 90 degrees
- moved R77 412.8 mm to (223.2, 186.3), turned to 90 degrees
- moved TP10 405.3 mm to (236.9, 184.0)
- moved R22 397.8 mm to (238.2, 185.8), turned to 90 degrees
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Connections:
- net +1V1 renamed /Keyboard/DVDD_L
- ACFET1 pad 5: /Charging IC/ADAPTER+ -> /usbC_Switcher/VBUS
- ACFET1 pad 6: /Charging IC/ADAPTER+ -> /usbC_Switcher/VBUS
- ACFET1 pad 7: /Charging IC/ADAPTER+ -> /usbC_Switcher/VBUS
- ACFET1 pad 8: /Charging IC/ADAPTER+ -> /usbC_Switcher/VBUS
- C50 pad 1: /Charging IC/ADAPTER+ -> /usbC_Switcher/VBUS
- D126 pad 1: /Charging IC/ADAPTER+ -> /usbC_Switcher/VBUS
- D128 pad 1: /usbC_Switcher/CC1 -> /usbC_Switcher/CC2
- J16 pad S1: (no net) -> GND
- J16 pad S2: (no net) -> GND
- J4 pad P1: (no net) -> GND
- J4 pad P2: (no net) -> GND
- J6 pad SH1: (no net) -> GND
- J6 pad SH2: (no net) -> GND
- L2 pad 2: Net-(L2-Pad2) -> +10V
- M1 pad SH1: (no net) -> GND
- M1 pad SH2: (no net) -> GND
- M2 pad 1: unconnected-(M2-D-Pad1) -> Net-(M3-S)
- M2 pad 2: unconnected-(M2-D-Pad2) -> Net-(M3-S)
- M3 pad 5: unconnected-(M3-D-Pad5) -> /VRM/voltIn
- M3 pad 6: unconnected-(M3-D-Pad6) -> /VRM/voltIn
- Q9 pad 1: /Charging IC/ACN -> /VRM/voltIn
- Q9 pad 2: Net-(Q9-G) -> /VRM/voltIn
- Q9 pad 4: (no net) -> Net-(Q9-G)
- Q9 pad 5: (no net) -> /Charging IC/ACN
- R50 pad 1: /Charging IC/ADAPTER+ -> /usbC_Switcher/VBUS
- R69 pad 1: /Charging IC/ADAPTER+ -> /usbC_Switcher/VBUS
- R70 pad 1: /Charging IC/ADAPTER+ -> /usbC_Switcher/VBUS
- Rcomp2 pad 2: Net-(L2-Pad2) -> +10V
- S13 pad 1: Net-(S13-Pad1) -> /Keyboard/Col_12
- S26 pad 1: Net-(S13-Pad1) -> /Keyboard/Col_12
- S39 pad 1: Net-(S13-Pad1) -> /Keyboard/Col_12
- S52 pad 1: Net-(S13-Pad1) -> /Keyboard/Col_12
- S65 pad 1: Net-(S13-Pad1) -> /Keyboard/Col_12
- S78 pad 1: Net-(S13-Pad1) -> /Keyboard/Col_12
- S91 pad 1: Net-(S13-Pad1) -> /Keyboard/Col_12
- U6 pad 25: unconnected-(U6-EPAD-Pad25) -> GND
Routing:
- net /Keyboard/Row_4: track 0.00 -> 754.0 mm, vias 0 -> 7
- net /Keyboard/Col_0: track 0.00 -> 579.3 mm, vias 0 -> 3
- net /Keyboard/Row_7: track 0.00 -> 562.8 mm, vias 0 -> 15
- net /Keyboard/Col_1: track 0.00 -> 539.7 mm, vias 0 -> 6
- net /Keyboard/Col_4: track 0.00 -> 520.6 mm, vias 0 -> 9
- net /Keyboard/Row_6: track 0.00 -> 513.4 mm, vias 0 -> 12
- net /Keyboard/Col_2: track 0.00 -> 503.1 mm, vias 0 -> 2
- net /Keyboard/Col_7: track 0.00 -> 498.5 mm, vias 0 -> 7
- net /Keyboard/Col_10: track 0.00 -> 483.1 mm, vias 0 -> 7
- net /Keyboard/Col_8: track 0.00 -> 482.2 mm, vias 0 -> 5
- net /Keyboard/Col_6: track 0.00 -> 463.0 mm, vias 0 -> 11
- net /Keyboard/Col_11: track 0.00 -> 456.9 mm, vias 0 -> 5
- net /Keyboard/Col_9: track 0.00 -> 437.3 mm, vias 0 -> 3
- net /Keyboard/Row_3: track 0.00 -> 408.3 mm, vias 0 -> 17
- net /Keyboard/Row_5: track 0.00 -> 405.7 mm, vias 0 -> 16
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- added copper zone on F.Cu, net +3V3
- added copper zone on B.Cu, net GND
Other:
- board size 49.6 x 53.5 mm -> 455.1 x 331.2 mm
