File: KiCad/RDAT/RDAT.kicad_pcb (KiCad board)
At the start: 4 copper layers, 455.2 x 254.8 mm, 520 parts, among them J1 Conn_01x02, J16 MDT420E03001, J2 Conn_01x02, J3 S8411-45R, J4 Bus_M.2_Socket_B, J5 USB_A_Stacked, J6 HDMI_A, J7 SF72S006VBDR2500, J8 MUSBRM1C130, M1 Fan_4pin, M2 CSD17571Q2, M3 CSD17571Q2, Q10 SI7135DP-T1-GE3, Q4 2N7002, Q5 2SK3018, Q6 2SK3018, Q7 2SK3018, Q8 2N7002, Q9 SI7135DP-T1-GE3, U1 W25Q128JVS, U11 CSD85302L, U12 LTC4412ES6#TRMPBF, U15 CH224K, U2 SC091413, U3 BQ7791500PWR, U4 BQ34Z100PWR-R2, U5 TPS54302, U6 BQ24617RGER, U7 TPS40345DRCR, U8 TPS54302, U9 CDDFN10-0524P, X1 ABM8-272-T3

Commit message: Generate Gerbers and Order PCB
Parts:
- C18: footprint Capacitor_SMD:C_0402_1005Metric -> Capacitor_SMD:C_0805_2012Metric
- C45, C46: footprint footprints:CAP-SMD_BD6.3-L6.6-W6.6-LS7.4-FD -> footprints:CAP-SMD_BD5.0-L5.3-W5.3-FD
- moved C18 4.46 mm to (465.4, 231.2), turned to 90 degrees
- moved C46 1.85 mm to (88.3, 186.9)
- moved C45 1.21 mm to (92.9, 181.0), turned to 180 degrees
Routing:
- net /~{PWR_LED}/~{PSON}: track 248.3 -> 393.6 mm, vias 4 -> 9
- net +3V3: track 924.3 -> 929.4 mm
- net Net-(U7-BP): track 3.52 -> 4.65 mm
- net GND: vias 1181 -> 1182
- removed copper zone on F.Cu, net +3V3
