File: KiCad/RDAT/B_key.kicad_sch (KiCad schematic)
At the start: 29 parts, among them J3 Conn_01x02, J4 Bus_M.2_Socket_B

Commit message: Placed a lot of components
Parts:
- removed C68: 100fP/50v, Capacitor_SMD:C_0402_1005Metric, symbol Device:C_Small
- removed J3: Conn_01x02, Connector_PinHeader_1.00mm:PinHeader_1x02_P1.00mm_Vertical, symbol Connector:SIM_Card
- added C73: 100fP/50v, Capacitor_SMD:C_0402_1005Metric, symbol Device:C_Small
- added J7: SF72S006VBDR2500, Connector_JAE:JAE_SIM_Card_SF72S006, symbol SF72S006VBDR2500:SF72S006VBDR2500
Connections:
- net GND: now also C73.1, J7.C5, J7.DSW, J7.GND1, J7.GND10, J7.GND2, J7.GND3, J7.GND4, J7.GND5, J7.GND6, J7.GND7, J7.GND8, J7.GND9
- net SIM_CLK: now also J7.C3
- net SIM_DATA: now also J7.C7
- net SIM_DET: now also J7.CSW
- net SIM_RST: now also J7.C2
- net VCC_SIM: now also J7.C1
- new net: C73.2, J7.C6
Other:
- moved on the sheet: D119, D120, D121, D122
