File: KiCad/RDAT/Charger.kicad_sch (KiCad schematic)
At the start: 58 parts, among them U6 BQ24617RGER

Commit message: End Of day commit
Parts:
- MOSFET2(Q4)1: footprint POWERPAK_1212-8 -> footprints:POWERPAK_1212-8_VIS
- U6: footprint RGE24_2P45X2P45 -> Package_DFN_QFN:Texas_RGE0024H_VQFN-24-1EP_4x4mm_P0.5mm_EP2.7x2.7mm_ThermalVias
Connections:
- net ACP: now also ACFET2.9 (D)
- net ADAPTER+: now also ACFET1.9 (D)
- net GND: now also U6.25 (EPAD)
- net PACK+: now also BATFET1.9 (D)
- net PH: now also MOSFET4(Q5)1.9 (D)
- net SYSTEM+: now also MOSFET2(Q4)1.9 (D)
Other:
- moved on the sheet: R_{AC}1
Changed lines of the file:
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@@
 	)
 	(junction
-		(at 90.17 111.76)
+		(at 130.81 109.22)
 		(diameter 0)
 		(color 0 0 0 0)
 	)
 	(junction
-		(at 35.56 50.8)
+		(at 90.17 111.76)
 		(diameter 0)
 		(color 0 0 0 0)
 	)
 	(junction
-		(at 151.13 173.99)
+		(at 35.56 50.8)
 		(diameter 0)
 		(color 0 0 0 0)
@@
 	)
 	(junction
+		(at 45.72 181.61)
+		(diameter 0)
+		(color 0 0 0 0)
+	)
+	(junction
 		(at 100.33 180.34)
 		(diameter 0)
@@
 	)
 	(junction
+		(at 59.69 120.65)
+		(diameter 0)
+		(color 0 0 0 0)
+	)
+	(junction
 		(at 156.21 116.84)
 		(diameter 0)
@@
 	)
 	(junction
+		(at 151.13 175.26)
+		(diameter 0)
+		(color 0 0 0 0)
+	)
+	(junction
 		(at 130.81 111.76)
 		(diameter 0)
@@
 		(color 0 0 0 0)
 	)
+	(junction
+		(at 195.58 118.11)
+		(diameter 0)
+		(color 0 0 0 0)
+	)
 	(wire
 		(pts
@@
 	(wire
 		(pts
-			(xy 151.13 177.8) (xy 148.59 177.8)
+			(xy 151.13 175.26) (xy 151.13 173.99)
 		)
 		(stroke
@@
 	(wire
 		(pts
-			(xy 151.13 177.8) (xy 151.13 173.99)
+			(xy 151.13 177.8) (xy 151.13 175.26)
 		)
 		(stroke
@@
 	(wire
 		(pts
+			(xy 45.72 175.26) (xy 46.99 175.26)
+		)
+		(stroke
+			(width 0)
+			(type default)
+		)
+	)
+	(wire
+		(pts
 			(xy 148.59 185.42) (xy 148.59 182.88)
 		)
@@
 	(wire
 		(pts
+			(xy 151.13 175.26) (xy 154.94 175.26)
+		)
+		(stroke
+			(width 0)
+			(type default)
+		)
+	)
+	(wire
+		(pts
 			(xy 57.15 50.8) (xy 58.42 50.8)
 		)
@@
 	(wire
 		(pts
-			(xy 90.17 111.76) (xy 90.17 114.3)
+			(xy 45.72 175.26) (xy 45.72 181.61)
 		)
 		(stroke
@@
 	(wire
 		(pts
-			(xy 175.26 116.84) (xy 180.34 116.84)
+			(xy 90.17 111.76) (xy 90.17 114.3)
 		)
 		(stroke
@@
 	(wire
 		(pts
-			(xy 38.1 78.74) (xy 38.1 97.79)
+			(xy 175.26 116.84) (xy 180.34 116.84)
 		)
 		(stroke
@@
 	(wire
 		(pts
-			(xy 154.94 173.99) (xy 151.13 173.99)
+			(xy 38.1 78.74) (xy 38.1 97.79)
 		)
 		(stroke
@@
 	(wire
 		(pts
-			(xy 44.45 181.61) (xy 46.99 181.61)
+			(xy 160.02 175.26) (xy 160.02 173.99)
+		)
+		(stroke
+			(width 0)
+			(type default)
+		)
+	)
+	(wire
+		(pts
+			(xy 44.45 181.61) (xy 45.72 181.61)
 		)
 		(stroke
@@
 	(wire
 		(pts
+			(xy 154.94 38.1) (xy 144.78 38.1)
+		)
+		(stroke
+			(width 0)
+			(type default)
+		)
+	)
+	(wire
+		(pts
 			(xy 95.25 189.23) (xy 95.25 193.04)
 		)
@@
 	(wire
 		(pts
+			(xy 148.59 175.26) (xy 148.59 177.8)
+		)
+		(stroke
+			(width 0)
+			(type default)
+		)
+	)
+	(wire
+		(pts
 			(xy 100.33 193.04) (xy 107.95 193.04)
 		)
@@
 	(wire
 		(pts
+			(xy 45.72 181.61) (xy 46.99 181.61)
+		)
+		(stroke
+			(width 0)
+			(type default)
+		)
+	)
+	(wire
+		(pts
 			(xy 147.32 116.84) (xy 156.21 116.84)
 		)
@@
 	(wire
 		(pts
+			(xy 198.12 123.19) (xy 198.12 118.11)
+		)
+		(stroke
+			(width 0)
+			(type default)
+		)
+	)
+	(wire
+		(pts
 			(xy 35.56 52.07) (xy 35.56 50.8)
 		)
@@
 	(wire
 		(pts
+			(xy 195.58 118.11) (xy 195.58 116.84)
+		)
+		(stroke
+			(width 0)
+			(type default)
+		)
+	)
+	(wire
+		(pts
 			(xy 200.66 55.88) (xy 200.66 57.15)
 		)
@@
 	(wire
 		(pts
-			(xy 195.58 123.19) (xy 195.58 116.84)
+			(xy 195.58 123.19) (xy 195.58 118.11)
+		)
+		(stroke
+			(width 0)
+			(type default)
+		)
+	)
+	(wire
+		(pts
+			(xy 130.81 106.68) (xy 130.81 109.22)
 		)
 		(stroke
@@
 	(wire
 		(pts
+			(xy 198.12 118.11) (xy 195.58 118.11)
+		)
+		(stroke
+			(width 0)
+			(type default)
+		)
+	)
+	(wire
+		(pts
 			(xy 46.99 185.42) (xy 46.99 182.88)
 		)
@@
 	(wire
 		(pts
+			(xy 59.69 118.11) (xy 59.69 120.65)
+		)
+		(stroke
+			(width 0)
+			(type default)
+		)
+	)
+	(wire
+		(pts
 			(xy 130.81 109.22) (xy 130.81 111.76)
 		)
@@
 	(wire
 		(pts
+			(xy 148.59 177.8) (xy 151.13 177.8)
+		)
+		(stroke
+			(width 0)
+			(type default)
+		)
+	)
+	(wire
+		(pts
 			(xy 176.53 162.56) (xy 176.53 163.83)
 		)
@@
 			)
 		)
-		(property "Footprint" "RGE24_2P45X2P45"
+		(property "Footprint" "Package_DFN_QFN:Texas_RGE0024H_VQFN-24-1EP_4x4mm_P0.5mm_EP2.7x2.7mm_ThermalVias"
 			(at 73.66 38.1 0)
 			(effects
@@
 			)
 		)
-		(property "Datasheet" "https://www.ti.com/cn/lit/gpn/bq24617"
+		(property "Datasheet" "https://www.ti.com/lit/ds/symlink/bq24610.pdf?HQS=dis-dk-null-digikeymode-dsf-pf-null-wwe&ts=1741164993119&ref_url=https%253A%252F%252Fwww.ti.com%252Fgeneral%252Fdocs%252Fsuppproductinfo.tsp%253FdistId%253D10%2526gotoUrl%253Dhttps%253A%252F%252Fwww.ti.com%252Flit%252Fgpn%252Fbq24610"
 			(at 73.66 38.1 0)
 			(effects
@@
 	)
 	(symbol
+		(lib_name "SIS412DN-T1-GE3_1")
 		(lib_id "SIS412DN:SIS412DN-T1-GE3")
 		(at 19.05 120.65 0)
@@
 			)
 		)
-		(property "Footprint" "POWERPAK_1212-8"
+		(property "Footprint" "footprints:POWERPAK_1212-8_VIS"
 			(at 19.05 120.65 0)
 			(effects
@@
 		(pin "3"
 		)
+		(pin "9"
+		)
 		(instances
 			(project "RDAT"
@@
 		(pin "4"
 		)
+		(pin "9"
+		)
 		(instances
 			(project "RDAT"
@@
 	(symbol
 		(lib_id "Device:R_Small_US")
-		(at 157.48 173.99 90)
+		(at 157.48 175.26 90)
 		(mirror x)
 		(unit 1)
@@
 		(dnp no)
 		(property "Reference" "R_{AC}1"
-			(at 160.274 176.276 90)
+			(at 160.274 177.546 90)
 			(effects
 				(font
@@
 		)
 		(property "Value" "0.01"
-			(at 165.1 176.276 90)
+			(at 165.1 177.546 90)
 			(effects
 				(font
@@
 		)
 		(property "Footprint" "footprints:RESC_WSHM2818R0150FEA"
-			(at 157.48 173.99 0)
+			(at 157.48 175.26 0)
 			(effects
 				(font
@@
 		)
 		(property "Datasheet" "https://wmsc.lcsc.com/wmsc/upload/file/pdf/v2/lcsc/2312131129_Vishay-Intertech-WSHP2818R0100FEA_C4274345.pdf"
-			(at 157.48 173.99 0)
+			(at 157.48 175.26 0)
 			(effects
 				(font
@@
 		)
 		(property "Description" "Resistor, small US symbol"
-			(at 157.48 173.99 0)
+			(at 157.48 175.26 0)
 			(effects
 				(font
@@
 		)
 		(property "JLCPCB_LINK" "https://jlcpcb.com/partdetail/VishayIntertech-WSHP2818R0100FEA/C4274345"
-			(at 157.48 173.99 0)
+			(at 157.48 175.26 0)
 			(effects
 				(font
@@
 		(pin "3"
 		)
+		(pin "9"
+		)
 		(instances
 			(project "RDAT"
@@
 	)
 	(symbol
+		(lib_id "power:GND")
+		(at 154.94 38.1 0)
+		(unit 1)
+		(exclude_from_sim no)
+		(in_bom yes)
+		(on_board yes)
+		(dnp no)
+		(fields_autoplaced yes)
+		(property "Reference" "#PWR090"
+			(at 154.94 44.45 0)
+			(effects
+				(font
+					(size 1.27 1.27)
+				)
+				(hide yes)
+			)
+		)
+		(property "Value" "GND"
+			(at 154.94 43.18 0)
+			(effects
+				(font
+					(size 1.27 1.27)
+				)
+			)
+		)
+		(property "Footprint" ""
+			(at 154.94 38.1 0)
+			(effects
+				(font
+					(size 1.27 1.27)
+				)
+				(hide yes)
+			)
+		)
+		(property "Datasheet" ""
+			(at 154.94 38.1 0)
+			(effects
+				(font
+					(size 1.27 1.27)
+				)
+				(hide yes)
+			)
+		)
+		(property "Description" "Power symbol creates a global label with name \"GND\" , ground"
+			(at 154.94 38.1 0)
+			(effects
+				(font
+					(size 1.27 1.27)
+				)
+				(hide yes)
+			)
+		)
+		(pin "1"
+		)
+		(instances
+			(project "RDAT"
+				(path "/0db9370a-8a21-4fd2-83a9-f207c3725dc9/64601ab1-4b63-421f-a3b9-e484b74e1409"
+					(reference "#PWR090")
+					(unit 1)
+				)
+			)
+		)
+	)
+	(symbol
 		(lib_id "Device:C_Small")
 		(at 200.66 43.18 0)
@@
 		(pin "6"
 		)
+		(pin "9"
+		)
 		(instances
 			(project "RDAT"
@@
 	)
 	(symbol
+		(lib_name "SI7617DN-T1-GE3_2")
 		(lib_id "SI7617DN-T1-GE3:SI7617DN-T1-GE3")
 		(at 87.63 177.8 0)
@@
 		(pin "4"
 		)
+		(pin "9"
+		)
 		(instances

Commit message: Most of the way thru routing
Parts:
- MOSFET4(Q5)1: footprint POWERPAK_1212-8 -> footprints:POWERPAK_1212-8_VIS
Changed lines of the file:
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@@
 			)
 		)
-		(property "Footprint" "POWERPAK_1212-8"
+		(property "Footprint" "footprints:POWERPAK_1212-8_VIS"
 			(at 90.17 109.22 0)
 			(effects
