File: KiCad/RDAT/Charger.kicad_sch (KiCad schematic)
At the start: 58 parts, among them U6 BQ24617RGER

Commit message: 2x checing of bom on JLCPCB
Parts:
- R107: value 68.1k/10% -> 68.1k; JLCPCB_PART_NUMBER (none) -> C11537
- R108: JLCPCB_PART_NUMBER (none) -> C25882
- R110: JLCPCB_PART_NUMBER (none) -> C25091
- R34: value 43k/10% -> 43k
- R35: value 5.1k/10% -> 5.1k
- R_{AC}1, R_{AC}2: JLCPCB_PART_NUMBER (none) -> C4274345
- R_{SR}1: value 0.01/1% -> 0.01; JLCPCB_PART_NUMBER (none) -> C4274345
- TH2: JLCPCB_PART_NUMBER (none) -> C13564
- U6: JLCPCB_PART_NUMBER (none) -> C914098

Commit message: Generate Gerbers and Order PCB
Parts:
- C40, C41: JLCPCB_LINK https://jlcpcb.com/partdetail/16204-CL05A106MQ5NUNC/C15525 -> https://jlcpcb.com/partdetail/97651-CL10A106MA8NRNC/C96446
- C45, C46: JLCPCB_LINK https://jlcpcb.com/partdetail/Roqang-RVT1E221M0607/C2918361 -> https://jlcpcb.com/partdetail/HonorElec-RVT1V100M0505/C30110
Changed lines of the file:
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@@
 			)
 		)
-		(property "JLCPCB_LINK" "https://jlcpcb.com/partdetail/Roqang-RVT1E221M0607/C2918361"
+		(property "JLCPCB_LINK" "https://jlcpcb.com/partdetail/HonorElec-RVT1V100M0505/C30110"
 			(at 181.61 177.8 0)
 			(effects
@@
 			)
 		)
-		(property "JLCPCB_LINK" "https://jlcpcb.com/partdetail/16204-CL05A106MQ5NUNC/C15525"
+		(property "JLCPCB_LINK" "https://jlcpcb.com/partdetail/97651-CL10A106MA8NRNC/C96446"
 			(at 156.21 119.38 0)
 			(effects
@@
 			)
 		)
-		(property "JLCPCB_LINK" "https://jlcpcb.com/partdetail/Roqang-RVT1E221M0607/C2918361"
+		(property "JLCPCB_LINK" "https://jlcpcb.com/partdetail/HonorElec-RVT1V100M0505/C30110"
 			(at 176.53 177.8 0)
 			(effects
@@
 			)
 		)
-		(property "JLCPCB_LINK" "https://jlcpcb.com/partdetail/16204-CL05A106MQ5NUNC/C15525"
+		(property "JLCPCB_LINK" "https://jlcpcb.com/partdetail/97651-CL10A106MA8NRNC/C96446"
 			(at 160.02 119.38 0)
 			(effects
