File: KiCad/RDAT/VRM.kicad_sch (KiCad schematic)
At the start: 63 parts, among them M2 CSD17571Q2, M3 CSD17571Q2, Q3 SI7135DP-T1-GE3, Q8 2N7002, Q9 SI7135DP-T1-GE3, U12 LTC4412ES6#TRMPBF, U5 TPS54302, U7 TPS40345DRCR, U8 TPS54302

Commit message: End Of day commit
Parts:
- removed Q3: SI7135DP-T1-GE3, Package_SO:PowerPAK_SO-8_Single, symbol Simulation_SPICE:PMOS
- added Q10: SI7135DP-T1-GE3, Package_SO:PowerPAK_SO-8_Single, symbol Simulation_SPICE:PMOS
- M2, M3: footprint Package_SON:WSON-6-1EP_2x2mm_P0.65mm_EP1x1.6mm_ThermalVias -> footprints:DQK0006C
Connections:
- net +10V: now also L2.2, Rcomp2.2
- net BATT_PW_IN: now also Q10.5 (D)
- net USB_PW_IN: now also Q9.5 (D); no longer Q9.1 (D)
- net voltIn: now also M3.5 (D), M3.6 (D), Q9.1 (S), Q9.2 (S), Q10.1 (S), Q10.2 (S), Q10.3 (S)
- net at M2.1 (D): now also C55.2, L2.1, M2.2 (D), M2.5 (D), M2.6 (D), M3.4 (S), U7.8 (SW)
- net at R21.1, U12.4 (STAT): now also Q9.4 (G); no longer Q9.2 (G)
- net at U12.5 (GATE): now also Q10.4 (G)
- no-connect marks 7 -> 2
Other:
- moved on the sheet: Q9

Commit message: 2x checing of bom on JLCPCB
Parts:
- C22, C32: value 100nF/64mOhm -> 100nF
- C23, C48, C71: value 47uF/3.037mOhm -> 47uF
- C60: value 10uF/1mOhm -> 10uF
- C61: value 4.7uF/3.52mohm(ESR) -> 4.7uF
- C66, C69: value 1uF/16V -> 1uF
- C70: value 47pF/0Ohm -> 47pF
- C72: value 82pF/0Ohm -> 82pF
- R105: JLCPCB_PART_NUMBER (none) -> C423242
- R58, R60: value 100R/1% -> 100R
- R62: value 1K/1% -> 1K
- R63: value 10K/1% -> 10K
- R64: value 2.2K/1% -> 2.2K
- Rcomp2: JLCPCB_PART_NUMBER (none) -> C25087
- Rcomp3: JLCPCB_PART_NUMBER (none) -> C25100
- Rfbb1: JLCPCB_PART_NUMBER (none) -> C8369
- Rfbb2: JLCPCB_PART_NUMBER (none) -> C270617
- S104, S105: JLCPCB_PART_NUMBER (none) -> C318884
- U12: JLCPCB_PART_NUMBER (none) -> C459883
- U5, U8: JLCPCB_PART_NUMBER (none) -> C311983
- U7: JLCPCB_PART_NUMBER (none) -> C2658407
