File: KiCad/RDAT/bms.kicad_sch (KiCad schematic)
At the start: 33 parts, among them U11 CSD85302L, U3 BQ7791500PWR, U4 BQ34Z100PWR-R2

Commit message: End Of day commit
Parts:
- U4: footprint PW14_TEX -> footprints:PW14_TEX
Connections:
- no-connect marks 2 -> 16
Changed lines of the file:
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@@
 	)
 	(no_connect
+		(at 60.96 256.54)
+	)
+	(no_connect
+		(at 60.96 243.84)
+	)
+	(no_connect
+		(at 60.96 248.92)
+	)
+	(no_connect
+		(at 15.24 248.92)
+	)
+	(no_connect
+		(at 15.24 246.38)
+	)
+	(no_connect
+		(at 15.24 256.54)
+	)
+	(no_connect
 		(at 100.33 123.19)
 	)
 	(no_connect
+		(at 15.24 254)
+	)
+	(no_connect
+		(at 60.96 254)
+	)
+	(no_connect
+		(at 60.96 251.46)
+	)
+	(no_connect
+		(at 15.24 259.08)
+	)
+	(no_connect
+		(at 60.96 259.08)
+	)
+	(no_connect
 		(at 100.33 107.95)
 	)
+	(no_connect
+		(at 60.96 246.38)
+	)
+	(no_connect
+		(at 15.24 251.46)
+	)
+	(no_connect
+		(at 15.24 243.84)
+	)
 	(wire
 		(pts
@@
 			)
 		)
-		(property "Footprint" "PW14_TEX"
+		(property "Footprint" "footprints:PW14_TEX"
 			(at 15.24 243.84 0)
 			(effects

Commit message: 2x checing of bom on JLCPCB
Parts:
- C17, C58, C59, C62, C63: value 1uF/10% -> 1uF
- R13: value 10k±1% -> 10k
- R85: value 1k/5% -> 1k; JLCPCB_PART_NUMBER (none) -> C11702
- R_{CHG}1: value 220/5% -> 220; JLCPCB_PART_NUMBER (none) -> C25091
- R_{DSG}1: value 470/5% -> 470; JLCPCB_PART_NUMBER (none) -> C25117
- R_{GS}1, R_{GS}2, R_{SNS}1: JLCPCB_PART_NUMBER (none) -> C26091
- SW_{HibernateBattery}1: JLCPCB_PART_NUMBER (none) -> C2921576
- TH_103AT_1: footprint Resistor_SMD:R_0201_0603Metric -> Resistor_SMD:R_0603_1608Metric; JLCPCB_PART_NUMBER (none) -> C13564
- U11: JLCPCB_PART_NUMBER (none) -> C701748
- U3: JLCPCB_PART_NUMBER (none) -> C2876946
