File: KiCad/RDAT/mu_cm.kicad_sch (KiCad schematic)
At the start: 9 parts

Commit message: 2x checked all schematics
Connections:
- net USB_2_P3+: now also A1.81 (USB2_P3+); no longer A1.79 (USB2_P3-)
- net USB_2_P3-: now also A1.79 (USB2_P3-); no longer A1.70 (USB2_P4+)
- net USB_2_P4-: now reaches A1.72 (USB2_P4-)
- net USB_2_P2-: now reaches A1.73 (USB2_P2-)
- net USB_2_P2+: now reaches A1.75 (USB2_P2+)
- new net USB_2_P4+: A1.70 (USB2_P4+)

Commit message: Pre-Annotate FULL, add usb
Parts:
- A1: JLCPCB_LINK (none) -> https://jlcpcb.com/partdetail/TeConnectivity-23094111/C5163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
- BT17: value Battery_Cell -> 3v; JLCPCB_LINK (none) -> https://jlcpcb.com/partdetail/Keystone-103/C238065
Other:
- note removed: "3V"
Changed lines of the file:
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@@
 		)
 	)
-	(text "3V"
-		(exclude_from_sim no)
-		(at 171.704 51.816 0)
-		(effects
-			(font
-				(size 1.27 1.27)
-			)
-		)
-	)
 	(text "HPD pin of unused DDI/TCP port\nneeds to be pulled down"
 		(exclude_from_sim no)
@@
 			)
 		)
-		(property "Value" "Battery_Cell"
-			(at 180.34 43.18 90)
+		(property "Value" "3v"
+			(at 172.974 51.308 90)
 			(effects
 				(font
@@
 			)
 		)
-		(property "Datasheet" "~"
+		(property "Datasheet" "https://www.lcsc.com/datasheet/lcsc_datasheet_2210171730_Harwin-S8411-45R_C5199899.pdf"
 			(at 173.736 49.53 90)
 			(effects
@@
 			)
 		)
+		(property "JLCPCB_LINK" "https://jlcpcb.com/partdetail/Keystone-103/C238065"
+			(at 175.26 49.53 0)
+			(effects
+				(font
+					(size 1.27 1.27)
+				)
+				(hide yes)
+			)
+		)
 		(pin "1"
 		)
@@
 			)
 		)
+		(property "JLCPCB_LINK" ""
+			(at 91.44 252.73 0)
+			(effects
+				(font
+					(size 1.27 1.27)
+				)
+			)
+		)
 		(pin "1"
 		)
@@
 			)
 		)
+		(property "JLCPCB_LINK" ""
+			(at 91.44 290.83 0)
+			(effects
+				(font
+					(size 1.27 1.27)
+				)
+			)
+		)
 		(pin "1"
 		)
@@
 			)
 		)
+		(property "JLCPCB_LINK" ""
+			(at 212.09 307.34 0)
+			(effects
+				(font
+					(size 1.27 1.27)
+				)
+			)
+		)
 		(pin "1"
 		)
@@
 			)
 		)
+		(property "JLCPCB_LINK" ""
+			(at 181.61 262.89 0)
+			(effects
+				(font
+					(size 1.27 1.27)
+				)
+			)
+		)
 		(pin "1"
 		)
@@
 			)
 		)
+		(property "JLCPCB_LINK" ""
+			(at 187.96 262.89 0)
+			(effects
+				(font
+					(size 1.27 1.27)
+				)
+			)
+		)
 		(pin "1"
 		)
@@
 			)
 		)
-		(property "Datasheet" ""
+		(property "Datasheet" "https://www.mouser.com/datasheet/2/830/DFRobot_ProductOverview_LattePandaMuMicrox86Comput-3483961.pdf"
 			(at 135.89 186.69 0)
 			(effects
@@
 			)
 		)
+		(property "JLCPCB_LINK" "https://jlcpcb.com/partdetail/TeConnectivity-23094111/C5163334"
+			(at 135.89 196.85 0)
+			(effects
+				(font
+					(size 1.27 1.27)
+				)
+				(hide yes)
+			)
+		)
 		(pin "68"
 		)
@@
 			)
 		)
+		(property "JLCPCB_LINK" ""
+			(at 161.29 49.53 0)
+			(effects
+				(font
+					(size 1.27 1.27)
+				)
+			)
+		)
 		(pin "1"
 		)
@@
 			)
 		)
+		(property "JLCPCB_LINK" ""
+			(at 237.49 307.34 0)
+			(effects
+				(font
+					(size 1.27 1.27)
+				)
+			)
+		)

Commit message: Added Libs and DOCS
Parts:
- R22: JLCPCB_LINK (none) -> https://jlcpcb.com/partdetail/26487-0402WGF1002TCE/C25744
- R7: footprint (none) -> Resistor_SMD:R_0402_1005Metric; JLCPCB_LINK (none) -> https://jlcpcb.com/partdetail/12256-0402WGF1001TCE/C11702
- R76, R77: JLCPCB_LINK (none) -> https://jlcpcb.com/partdetail/26484-0402WGF1003TCE/C25741
Changed lines of the file:
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@@
 			)
 		)
-		(property "Datasheet" "~"
+		(property "Datasheet" "https://jlcpcb.com/api/file/downloadByFileSystemAccessId/8579705919464263680"
 			(at 91.44 252.73 0)
 			(effects
@@
 			)
 		)
-		(property "JLCPCB_LINK" ""
+		(property "JLCPCB_LINK" "https://jlcpcb.com/partdetail/26484-0402WGF1003TCE/C25741"
 			(at 91.44 252.73 0)
 			(effects
@@
 					(size 1.27 1.27)
 				)
+				(hide yes)
 			)
 		)
@@
 			)
 		)
-		(property "Datasheet" "~"
+		(property "Datasheet" "https://jlcpcb.com/api/file/downloadByFileSystemAccessId/8579705919464263680"
 			(at 91.44 290.83 0)
 			(effects
@@
 			)
 		)
-		(property "JLCPCB_LINK" ""
+		(property "JLCPCB_LINK" "https://jlcpcb.com/partdetail/26484-0402WGF1003TCE/C25741"
 			(at 91.44 290.83 0)
 			(effects
@@
 					(size 1.27 1.27)
 				)
+				(hide yes)
 			)
 		)
@@
 			)
 		)
-		(property "Datasheet" "~"
+		(property "Datasheet" "https://jlcpcb.com/api/file/downloadByFileSystemAccessId/8556212101498380288"
 			(at 187.96 262.89 0)
 			(effects
@@
 			)
 		)
-		(property "JLCPCB_LINK" ""
+		(property "JLCPCB_LINK" "https://jlcpcb.com/partdetail/26487-0402WGF1002TCE/C25744"
 			(at 187.96 262.89 0)
 			(effects
@@
 					(size 1.27 1.27)
 				)
+				(hide yes)
 			)
 		)
@@
 			)
 		)
-		(property "Footprint" ""
+		(property "Footprint" "Resistor_SMD:R_0402_1005Metric"
 			(at 161.544 48.514 90)
 			(effects
@@
 			)
 		)
-		(property "Datasheet" "~"
+		(property "Datasheet" "https://jlcpcb.com/api/file/downloadByFileSystemAccessId/8579705924167974912"
 			(at 161.29 49.53 0)
 			(effects
@@
 			)
 		)
-		(property "JLCPCB_LINK" ""
+		(property "JLCPCB_LINK" "https://jlcpcb.com/partdetail/12256-0402WGF1001TCE/C11702"
 			(at 161.29 49.53 0)
 			(effects
@@
 					(size 1.27 1.27)
 				)
-			)
-		)
+				(hide yes)
+			)
+		)

Commit message: Push before Board Layout
Parts:
- A1: footprint Module_LattePanda:LattePanda_Module_H8.0mm_Horizontal -> footprints:LattePanda_Module_H4.0mm_Horizontal
- BT17: footprint A_HDJ_Library:Battery_Holder_CR1220_S8411-45R -> footprints:HARWIN_S8411-45R; JLCPCB_LINK https://jlcpcb.com/partdetail/Keystone-103/C238065 -> https://jlcpcb.com/partdetail/Harwin-S841145R/C5199899
- H5, H6: footprint A_HDJ_Library:MountingHole_3mm_M2_Pad_TopOnly -> MountingHole:MountingHole_2.2mm_M2_Pad_TopBottom
- R22, R76, R77: footprint A_HDJ_Library:R_0402_1005Metric -> Resistor_SMD:R_0402_1005Metric
- TP10: footprint A_HDJ_Library:TestPoint_Pad_D1.5mm -> TestPoint:TestPoint_Pad_D1.0mm
Changed lines of the file:
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@@
 			)
 		)
-		(property "Footprint" "A_HDJ_Library:Battery_Holder_CR1220_S8411-45R"
+		(property "Footprint" "footprints:HARWIN_S8411-45R"
 			(at 173.736 49.53 90)
 			(effects
@@
 			)
 		)
-		(property "JLCPCB_LINK" "https://jlcpcb.com/partdetail/Keystone-103/C238065"
+		(property "JLCPCB_LINK" "https://jlcpcb.com/partdetail/Harwin-S841145R/C5199899"
 			(at 175.26 49.53 0)
 			(effects
@@
 			)
 		)
-		(property "Footprint" "A_HDJ_Library:R_0402_1005Metric"
+		(property "Footprint" "Resistor_SMD:R_0402_1005Metric"
 			(at 91.44 250.952 90)
 			(effects
@@
 			)
 		)
-		(property "Footprint" "A_HDJ_Library:R_0402_1005Metric"
+		(property "Footprint" "Resistor_SMD:R_0402_1005Metric"
 			(at 91.44 289.052 90)
 			(effects
@@
 			)
 		)
-		(property "Footprint" "A_HDJ_Library:MountingHole_3mm_M2_Pad_TopOnly"
+		(property "Footprint" "MountingHole:MountingHole_2.2mm_M2_Pad_TopBottom"
 			(at 212.09 307.34 0)
 			(effects
@@
 			)
 		)
-		(property "Footprint" "A_HDJ_Library:TestPoint_Pad_D1.5mm"
+		(property "Footprint" "TestPoint:TestPoint_Pad_D1.0mm"
 			(at 186.69 262.89 0)
 			(effects
@@
 			)
 		)
-		(property "Footprint" "A_HDJ_Library:R_0402_1005Metric"
+		(property "Footprint" "Resistor_SMD:R_0402_1005Metric"
 			(at 187.96 264.668 90)
 			(effects
@@
 			)
 		)
-		(property "Footprint" "Module_LattePanda:LattePanda_Module_H8.0mm_Horizontal"
+		(property "Footprint" "footprints:LattePanda_Module_H4.0mm_Horizontal"
 			(at 135.89 186.69 0)
 			(effects
@@
 			)
 		)
-		(property "Footprint" "A_HDJ_Library:MountingHole_3mm_M2_Pad_TopOnly"
+		(property "Footprint" "MountingHole:MountingHole_2.2mm_M2_Pad_TopBottom"
 			(at 237.49 307.34 0)
 			(effects

Commit message: End Of day commit
Parts:
- removed BT17: 3v, footprints:HARWIN_S8411-45R, symbol Device:Battery_Cell
- added J3: S8411-45R, footprints:HARWIN_S8411-45R, symbol S8411-45R:S8411-45R
Connections:
- net GND: now also J3.N
- net at R7.2: now also J3.P
- no-connect marks 47 -> 110

Commit message: push prior to autorouting
Connections:
- net VPullup renamed +3V3
- no-connect marks 110 -> 112
Changed lines of the file:
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@@
+	)
+	(no_connect
+		(at 95.25 209.55)
 	)
 	(no_connect
@@
 	(no_connect
 		(at 176.53 313.69)
+	)
+	(no_connect
+		(at 95.25 207.01)
 	)
 	(no_connect
@@
 	)
 	(symbol
+		(lib_id "power:+3V3")
+		(at 196.85 262.89 0)
+		(unit 1)
+		(exclude_from_sim no)
+		(in_bom yes)
+		(on_board yes)
+		(dnp no)
+		(fields_autoplaced yes)
+		(property "Reference" "#PWR02"
+			(at 196.85 266.7 0)
+			(effects
+				(font
+					(size 1.27 1.27)
+				)
+				(hide yes)
+			)
+		)
+		(property "Value" "+3V3"
+			(at 196.85 257.81 0)
+			(effects
+				(font
+					(size 1.27 1.27)
+				)
+			)
+		)
+		(property "Footprint" ""
+			(at 196.85 262.89 0)
+			(effects
+				(font
+					(size 1.27 1.27)
+				)
+				(hide yes)
+			)
+		)
+		(property "Datasheet" ""
+			(at 196.85 262.89 0)
+			(effects
+				(font
+					(size 1.27 1.27)
+				)
+				(hide yes)
+			)
+		)
+		(property "Description" "Power symbol creates a global label with name \"+3V3\""
+			(at 196.85 262.89 0)
+			(effects
+				(font
+					(size 1.27 1.27)
+				)
+				(hide yes)
+			)
+		)
+		(pin "1"
+		)
+		(instances
+			(project ""
+				(path "/0db9370a-8a21-4fd2-83a9-f207c3725dc9/5b2d2e6c-036c-404a-b71b-c732d724c5c0"
+					(reference "#PWR02")
+					(unit 1)
+				)
+			)
+		)
+	)
+	(symbol
 		(lib_id "power:GND")
 		(at 87.63 252.73 270)
@@
 					(unit 1)
 				)
-			)
-		)
-	)
-	(symbol
-		(lib_name "+3V3_1")
-		(lib_id "power:+3V3")
-		(at 196.85 262.89 270)
-		(unit 1)
-		(exclude_from_sim no)
-		(in_bom yes)
-		(on_board yes)
-		(dnp no)
-		(fields_autoplaced yes)
-		(property "Reference" "#PWR019"
-			(at 193.04 262.89 0)
-			(effects
-				(font
-					(size 1.27 1.27)
-				)
-				(hide yes)
-			)
-		)
-		(property "Value" "VPullup"
-			(at 200.66 262.8899 90)
-			(effects
-				(font
-					(size 1.27 1.27)
-				)
-				(justify left)
-			)
-		)
-		(property "Footprint" ""
-			(at 196.85 262.89 0)
-			(effects
-				(font
-					(size 1.27 1.27)
-				)
-				(hide yes)
-			)
-		)
-		(property "Datasheet" ""
-			(at 196.85 262.89 0)
-			(effects
-				(font
-					(size 1.27 1.27)
-				)
-				(hide yes)
-			)
-		)
-		(property "Description" "Power symbol creates a global label with name \"VPullup\""
-			(at 196.85 262.89 0)
-			(effects
-				(font
-					(size 1.27 1.27)
-				)
-				(hide yes)
-			)
-		)
-		(pin "1"
-		)
-		(instances
-			(project "RDAT"
-				(path "/0db9370a-8a21-4fd2-83a9-f207c3725dc9/5b2d2e6c-036c-404a-b71b-c732d724c5c0"
-					(reference "#PWR019")
-					(unit 1)
-				)

Commit message: Adequitely Passing DRC
Connections:
- net GND: now also A1.101 (GND), A1.107 (GND), A1.11 (GND), A1.110 (GND), A1.113 (GND), A1.116 (GND), A1.135 (GND), A1.136 (GND), A1.14 (GND), A1.151 (GND), A1.158 (GND), A1.167 (GND), A1.17 (GND), A1.170 (GND), A1.181 (GND), A1.182 (GND), A1.188 (GND), A1.189 (GND), A1.194 (GND), A1.195 (GND), A1.20 (GND), A1.200 (GND), A1.201 (GND), A1.206 (GND), A1.207 (GND), A1.212 (GND), A1.213 (GND), A1.218 (GND), A1.219 (GND), A1.224 (GND), A1.225 (GND), A1.23 (GND), A1.230 (GND), A1.231 (GND), A1.236 (GND), A1.237 (GND), A1.242 (GND), A1.243 (GND), A1.248 (GND), A1.249 (GND), A1.26 (GND), A1.29 (GND), A1.32 (GND), A1.35 (GND), A1.38 (GND), A1.41 (GND), A1.44 (GND), A1.47 (GND), A1.50 (GND), A1.53 (GND), A1.56 (GND), A1.59 (GND), A1.62 (GND), A1.65 (GND), A1.68 (GND), A1.71 (GND), A1.74 (GND), A1.77 (GND), A1.80 (GND), A1.83 (GND), A1.86 (GND), A1.89 (GND), A1.92 (GND), A1.95 (GND), A1.98 (GND), A1.MP (Mountinge_Pads)
- no-connect marks 112 -> 136
Changed lines of the file:
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@@
+	)
+	(junction
+		(at 134.62 331.47)
+		(diameter 0)
+		(color 0 0 0 0)
 	)
 	(junction
@@
 	)
 	(no_connect
+		(at 95.25 267.97)
+	)
+	(no_connect
 		(at 176.53 99.06)
 	)
@@
 	)
 	(no_connect
+		(at 95.25 280.67)
+	)
+	(no_connect
 		(at 176.53 160.02)
 	)
@@
 	)
 	(no_connect
+		(at 95.25 300.99)
+	)
+	(no_connect
 		(at 176.53 292.1)
 	)
 	(no_connect
+		(at 95.25 316.23)
+	)
+	(no_connect
 		(at 176.53 287.02)
 	)
@@
 	)
 	(no_connect
+		(at 95.25 308.61)
+	)
+	(no_connect
 		(at 95.25 105.41)
 	)
 	(no_connect
+		(at 95.25 262.89)
+	)
+	(no_connect
+		(at 95.25 273.05)
+	)
+	(no_connect
 		(at 95.25 97.79)
 	)
@@
 	)
 	(no_connect
+		(at 95.25 275.59)
+	)
+	(no_connect
 		(at 176.53 267.97)
 	)
@@
 	)
 	(no_connect
+		(at 95.25 297.18)
+	)
+	(no_connect
 		(at 95.25 80.01)
 	)
@@
 	)
 	(no_connect
+		(at 95.25 323.85)
+	)
+	(no_connect
 		(at 95.25 148.59)
 	)
@@
 	)
 	(no_connect
+		(at 95.25 321.31)
+	)
+	(no_connect
 		(at 176.53 189.23)
 	)
@@
 	)
 	(no_connect
+		(at 95.25 311.15)
+	)
+	(no_connect
 		(at 95.25 135.89)
 	)
@@
 	)
 	(no_connect
+		(at 95.25 285.75)
+	)
+	(no_connect
 		(at 176.53 130.81)
 	)
@@
 	)
 	(no_connect
+		(at 95.25 278.13)
+	)
+	(no_connect
 		(at 176.53 252.73)
 	)
@@
 	)
 	(no_connect
+		(at 95.25 306.07)
+	)
+	(no_connect
 		(at 95.25 146.05)
 	)
@@
 	)
 	(no_connect
+		(at 95.25 294.64)
+	)
+	(no_connect
 		(at 176.53 313.69)
 	)
@@
 	)
 	(no_connect
+		(at 95.25 259.08)
+	)
+	(no_connect
 		(at 176.53 165.1)
 	)
@@
 	)
 	(no_connect
+		(at 95.25 270.51)
+	)
+	(no_connect
+		(at 95.25 256.54)
+	)
+	(no_connect
 		(at 95.25 179.07)
 	)
@@
 	)
 	(no_connect
+		(at 95.25 265.43)
+	)
+	(no_connect
 		(at 176.53 222.25)
 	)
@@
 	)
 	(no_connect
+		(at 95.25 283.21)
+	)
+	(no_connect
+		(at 95.25 318.77)
+	)
+	(no_connect
 		(at 176.53 273.05)
 	)
@@
 	)
 	(no_connect
+		(at 95.25 313.69)
+	)
+	(no_connect
 		(at 95.25 158.75)
 	)
@@
 	)
 	(no_connect
+		(at 95.25 303.53)
+	)
+	(no_connect
 		(at 176.53 304.8)
 	)
@@
 	(wire
 		(pts
+			(xy 134.62 331.47) (xy 135.89 331.47)
+		)
+		(stroke
+			(width 0)
+			(type default)
+		)
+	)
+	(wire
+		(pts
 			(xy 63.5 214.63) (xy 95.25 214.63)
 		)
@@
 		(pts
 			(xy 74.93 118.11) (xy 95.25 118.11)
+		)
+		(stroke
+			(width 0)
+			(type default)
+		)
+	)
+	(wire
+		(pts
+			(xy 133.35 331.47) (xy 134.62 331.47)
 		)
 		(stroke
@@
 					(unit 1)
 				)
+			)
+		)
+	)
+	(symbol
+		(lib_id "power:GND")
+		(at 134.62 331.47 0)
+		(unit 1)
+		(exclude_from_sim no)
+		(in_bom yes)
+		(on_board yes)
+		(dnp no)
+		(fields_autoplaced yes)
+		(property "Reference" "#PWR019"
+			(at 134.62 337.82 0)
+			(effects
+				(font
+					(size 1.27 1.27)
+				)
+				(hide yes)
+			)
+		)
+		(property "Value" "GND"
+			(at 134.62 336.55 0)
+			(effects
+				(font
+					(size 1.27 1.27)
+				)
+			)
+		)
+		(property "Footprint" ""
+			(at 134.62 331.47 0)
+			(effects
+				(font
+					(size 1.27 1.27)
+				)
+				(hide yes)
+			)
+		)
+		(property "Datasheet" ""
+			(at 134.62 331.47 0)
+			(effects
+				(font
+					(size 1.27 1.27)
+				)
+				(hide yes)
+			)
+		)
+		(property "Description" "Power symbol creates a global label with name \"GND\" , ground"
+			(at 134.62 331.47 0)
+			(effects
+				(font
+					(size 1.27 1.27)
+				)
+				(hide yes)
+			)
+		)
+		(pin "1"
+		)
+		(instances
+			(project ""
+				(path "/0db9370a-8a21-4fd2-83a9-f207c3725dc9/5b2d2e6c-036c-404a-b71b-c732d724c5c0"
+					(reference "#PWR019")
+					(unit 1)
+				)

Commit message: 2x checing of bom on JLCPCB
Parts:
- R22: value 10K/1% -> 10K
- R7: value 1K/1% -> 1K
- R76, R77: value 100K/1% -> 100K; JLCPCB_PART_NUMBER (none) -> C25741
Changed lines of the file:
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@@
 			)
 		)
-		(property "Value" "100K/1%"
+		(property "Value" "100K"
 			(at 91.948 255.27 90)
 			(effects
@@
 				)
 				(hide yes)
+			)
+		)
+		(property "JLCPCB_PART_NUMBER" "C25741"
+			(at 91.44 252.73 0)
+			(effects
+				(font
+					(size 1.27 1.27)
+				)
 			)
 		)
@@
 			)
 		)
-		(property "Value" "100K/1%"
+		(property "Value" "100K"
 			(at 91.948 293.37 90)
 			(effects
@@
 				)
 				(hide yes)
+			)
+		)
+		(property "JLCPCB_PART_NUMBER" "C25741"
+			(at 91.44 290.83 0)
+			(effects
+				(font
+					(size 1.27 1.27)
+				)
 			)
 		)
@@
 			)
 		)
+		(property "JLCPCB_PART_NUMBER" ""
+			(at 212.09 307.34 0)
+			(effects
+				(font
+					(size 1.27 1.27)
+				)
+			)
+		)
 		(pin "1"
 		)
@@
 			)
 		)
+		(property "JLCPCB_PART_NUMBER" ""
+			(at 181.61 262.89 0)
+			(effects
+				(font
+					(size 1.27 1.27)
+				)
+			)
+		)
 		(pin "1"
 		)
@@
 			)
 		)
-		(property "Value" "10K/1%"
+		(property "Value" "10K"
 			(at 191.262 267.208 90)
 			(effects
@@
 				)
 				(hide yes)
+			)
+		)
+		(property "JLCPCB_PART_NUMBER" ""
+			(at 187.96 262.89 0)
+			(effects
+				(font
+					(size 1.27 1.27)
+				)
 			)
 		)
@@
 			)
 		)
+		(property "JLCPCB_PART_NUMBER" ""
+			(at 177.8 49.53 0)
+			(effects
+				(font
+					(size 1.27 1.27)
+				)
+			)
+		)
 		(pin "N"
 		)
@@
 			)
 		)
+		(property "JLCPCB_PART_NUMBER" ""
+			(at 135.89 196.85 0)
+			(effects
+				(font
+					(size 1.27 1.27)
+				)
+			)
+		)
 		(pin "68"
 		)
@@
 			)
 		)
-		(property "Value" "1K/1%"
+		(property "Value" "1K"
 			(at 161.29 45.72 90)
 			(effects
@@
 				)
 				(hide yes)
+			)
+		)
+		(property "JLCPCB_PART_NUMBER" ""
+			(at 161.29 49.53 0)
+			(effects
+				(font
+					(size 1.27 1.27)
+				)
 			)
 		)
@@
 			(at 237.49 307.34 0)
 			(effects
+				(font
+					(size 1.27 1.27)
+				)
+			)
+		)
+		(property "JLCPCB_PART_NUMBER" ""
+			(at 237.49 307.34 0)
+			(effects
