File: KiCad/RDAT/E_Key.kicad_sch (KiCad schematic)
At the start: 12 parts, among them J16 MDT420E03001

Commit message: 2x checing of bom on JLCPCB
Parts:
- C80, C81: value 220nF/50V -> 220nF
- C82, C84: value 10uF/10V -> 10uF
- C83, C85: value 100nF/50V -> 100nF
- R72, R73: value 0R/1% -> 0R; JLCPCB_PART_NUMBER (none) -> C17168
- R74, R75: value 10K/1% -> 10K
Changed lines of the file:
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@@
 			)
 		)
-		(property "Value" "220nF/50V"
+		(property "Value" "220nF"
 			(at 78.74 83.82 90)
 			(effects
@@
 				)
 				(hide yes)
+			)
+		)
+		(property "JLCPCB_PART_NUMBER" ""
+			(at 77.47 85.09 0)
+			(effects
+				(font
+					(size 1.27 1.27)
+				)
 			)
 		)
@@
 			)
 		)
-		(property "Value" "220nF/50V"
+		(property "Value" "220nF"
 			(at 78.74 86.36 90)
 			(effects
@@
 				)
 				(hide yes)
+			)
+		)
+		(property "JLCPCB_PART_NUMBER" ""
+			(at 77.47 87.63 0)
+			(effects
+				(font
+					(size 1.27 1.27)
+				)
 			)
 		)
@@
 			)
 		)
-		(property "Value" "10K/1%"
+		(property "Value" "10K"
 			(at 177.8 95.25 0)
 			(effects
@@
 				)
 				(hide yes)
+			)
+		)
+		(property "JLCPCB_PART_NUMBER" ""
+			(at 179.07 93.98 0)
+			(effects
+				(font
+					(size 1.27 1.27)
+				)
 			)
 		)
@@
 			)
 		)
-		(property "Value" "10uF/10V"
+		(property "Value" "10uF"
 			(at 149.86 55.88 90)
 			(effects
@@
 				)
 				(hide yes)
+			)
+		)
+		(property "JLCPCB_PART_NUMBER" ""
+			(at 143.51 57.15 0)
+			(effects
+				(font
+					(size 1.27 1.27)
+				)
 			)
 		)
@@
 			)
 		)
-		(property "Value" "10uF/10V"
+		(property "Value" "10uF"
 			(at 149.86 43.18 90)
 			(effects
@@
 				)
 				(hide yes)
+			)
+		)
+		(property "JLCPCB_PART_NUMBER" ""
+			(at 143.51 44.45 0)
+			(effects
+				(font
+					(size 1.27 1.27)
+				)
 			)
 		)
@@
 			)
 		)
+		(property "JLCPCB_PART_NUMBER" ""
+			(at 137.16 118.11 0)
+			(effects
+				(font
+					(size 1.27 1.27)
+				)
+			)
+		)
 		(pin "5"
 		)
@@
 			)
 		)
-		(property "Value" "0R/1%"
+		(property "Value" "0R"
 			(at 173.99 147.32 90)
 			(effects
@@
 				)
 				(hide yes)
+			)
+		)
+		(property "JLCPCB_PART_NUMBER" "C17168"
+			(at 177.8 146.05 0)
+			(effects
+				(font
+					(size 1.27 1.27)
+				)
 			)
 		)
@@
 			)
 		)
-		(property "Value" "0R/1%"
+		(property "Value" "0R"
 			(at 109.22 60.96 0)
 			(effects
@@
 				)
 				(hide yes)
+			)
+		)
+		(property "JLCPCB_PART_NUMBER" "C17168"
+			(at 101.6 62.23 0)
+			(effects
+				(font
+					(size 1.27 1.27)
+				)
 			)
 		)
@@
 			)
 		)
+		(property "JLCPCB_PART_NUMBER" ""
+			(at 25.4 92.71 0)
+			(effects
+				(font
+					(size 1.27 1.27)
+				)
+			)
+		)
 		(pin "1"
 		)
@@
 			)
 		)
-		(property "Value" "100nF/50V"
+		(property "Value" "100nF"
 			(at 149.86 62.23 90)
 			(effects
@@
 				)
 				(hide yes)
+			)
+		)
+		(property "JLCPCB_PART_NUMBER" ""
+			(at 143.51 63.5 0)
+			(effects
+				(font
+					(size 1.27 1.27)
+				)
 			)
 		)
@@
 			)
 		)
-		(property "Value" "100nF/50V"
+		(property "Value" "100nF"
 			(at 149.86 49.53 90)
 			(effects
@@
 				)
 				(hide yes)
+			)
+		)
+		(property "JLCPCB_PART_NUMBER" ""
+			(at 143.51 50.8 0)
+			(effects
+				(font
+					(size 1.27 1.27)
+				)
 			)
 		)
@@
 			)
 		)
-		(property "Value" "10K/1%"
+		(property "Value" "10K"
 			(at 184.15 92.71 0)
 			(effects
@@
 			)
 		)
+		(property "JLCPCB_PART_NUMBER" ""
+			(at 182.88 93.98 0)
+			(effects
+				(font
+					(size 1.27 1.27)
+				)
+			)
+		)

Commit message: Generate Gerbers and Order PCB
Parts:
- C82, C84: JLCPCB_LINK https://jlcpcb.com/partdetail/16204-CL05A106MQ5NUNC/C15525 -> https://jlcpcb.com/partdetail/97651-CL10A106MA8NRNC/C96446
Changed lines of the file:
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@@
 			)
 		)
-		(property "JLCPCB_LINK" "https://jlcpcb.com/partdetail/16204-CL05A106MQ5NUNC/C15525"
+		(property "JLCPCB_LINK" "https://jlcpcb.com/partdetail/97651-CL10A106MA8NRNC/C96446"
 			(at 143.51 57.15 0)
 			(effects
@@
 			)
 		)
-		(property "JLCPCB_LINK" "https://jlcpcb.com/partdetail/16204-CL05A106MQ5NUNC/C15525"
+		(property "JLCPCB_LINK" "https://jlcpcb.com/partdetail/97651-CL10A106MA8NRNC/C96446"
 			(at 143.51 44.45 0)
 			(effects
